File: ReST Mainboard/_saved_ReST.sch (KiCad schematic (older format))
At the start: 87 parts

Commit message: Added PDF
Parts:
- added P? (x4): CONN_01X03, symbol CONN_01X03
Connections:
- net labels added: SERVO1, SERVO2, SERVO3, SERVO4
- wire segments 505 -> 413
