File: ReST Mainboard/_saved_ReST.sch (KiCad schematic (older format))
At the start: 92 parts

Commit message: Changed Additional-Board and Pinout
Sooo... I thought adding multiple Additional Module Boards would be bit much. Looked back at some older projects of mine and thought that using something like the uln2803 would be pretty neat (like 8 NPN Transitors, each 500mah and that in a DIL-18 Package IIRC) Which turns price really down, aswell as the size of the module. 
But using that one resultet in removing many extra pinouts, leaving with only 5 unused pins which will be broken out extra. This may change when the lcd pinout is finished. adding extra pinout for the additional board could also work out (as it occupies 8 pwm pins). I will look to copy that all into the schematic

Also missing: I2C EEPROM/Flash for settings
Parts:
- removed P?: CONN_02X06, symbol CONN_02X06
- added P? (x4): CONN_01X04, symbol CONN_01X04
- added P?: CONN_02X06, symbol CONN_02X06
- added P?: CONN_02X09, symbol CONN_02X09
Connections:
- net labels added: EXTRA1, EXTRA10, EXTRA11, EXTRA12, EXTRA2, EXTRA3, EXTRA4, EXTRA5, EXTRA6, EXTRA7, EXTRA8, EXTRA9, I2C1-SCL, I2C1-SDA, PWM-ADD, PWM-ADD0, PWM-ADD1, PWM-ADD2, PWM-ADD3, PWM-ADD4, PWM-ADD5, PWM-ADD6, PWM-ADD7, PWM-HEAT0, SPI2-EXTRA1, SPI2-EXTRA2, SPI2-MISO, SPI2-MOSI, SPI2-NSS, SPI2-SCK, SWCLK, SWDIO, UART1-RX, UART1-TX, UART5-RX, UART5-TX
- net labels removed: ADD, PWM-HEAT2
- wire segments 429 -> 456
