File: ReST Mainboard/_autosave-ReST.kicad_pcb (KiCad board)
At the start: 2 copper layers, 100 x 100 mm, 283 parts, among them IC1 AT24C128, P1 CONN_02X08, P10 CONN_01X04, P11 CONN_01X04, P12 CONN_02X04, P13 CONN_01X03, P14 CONN_02X03, P15 CONN_01X05, P16 CONN_01X03, P17 CONN_01X04, P18 CONN_02X04, P19 CONN_01X04, P2 CONN_02X08, P20 CONN_02X04, P21 CONN_02X04, P22 CONN_01X03, P23 SCREW_01X03, P24 CONN_01X03, P25 SCREW_01X03, P26 CONN_01X03, P27 SCREW_01X03, P28 CONN_01X03, P29 SCREW_01X03, P3 CONN_02X07, P30 CONN_01X03, P31 SCREW_01X03, P32 CONN_01X03, P33 SCREW_01X03, P34 CONN_01X03, P35 SCREW_01X04, P36 SCREW_01X04, P37 SCREW_01X04, P38 SCREW_01X04, P39 CONN_02X04, P4 CONN_02X10, P40 CONN_01X04, P41 CONN_01X04, P42 CONN_01X04, P43 CONN_02X03, P44 CONN_02X03, P45 CONN_02X03, P46 CONN_02X03, P5 USB_OTG, P6 CONN_02X05, P7 CONN_02X05, P8 CONN_01X09, P9 CONN_01X02, SW1 SW-SPST-NO, U1 STM32F103VE, U2 USBLC6-2, U3 L7805ACD2T-TR, U4 LM2574N-ADJ, U5 POLOLU_A4988, U6 POLOLU_A4988, U7 POLOLU_A4988, U8 POLOLU_A4988, X1 Crystal_Small

Commit message: Added BOM for all Items + suggested Links
Parts:
- removed 1111, 11111, 111111, 11111110, 11111111, 111111110, 111111111 (x2), 1111111110, 1111111111, 1111111112, 1111111113, 1111111114, 1111111115, 1111111116, 1111111117, 1111111118, 1111111119, 111111112 (x2), 1111111120, 111111113 (x2), 111111114 (x2), 111111115 (x2), 111111116, 111111117, 111111118, 111111119, 11111112 (x2), 111111121, 1111111210, 1111111211, 1111111212, 1111111213, 1111111214, 1111111215, 1111111216, 1111111217, 1111111218, 1111111219, 111111122, 1111111220, 111111123, 111111124, 111111125, 111111126, 111111127, 111111128, 111111129, 11111113 (x2), 111111131, 1111111310, 1111111311, 1111111312, 1111111313, 1111111314, 1111111315, 1111111316, 1111111317, 1111111318, 1111111319, 111111132, 1111111320, 111111133, 111111134, 111111135, 111111136, 111111137, 111111138, 111111139, 11111114 (x2), 11111115 (x2), 11111116, 11111117, 11111118, 11111119, 1111112, 11111121, 111111210, 111111211, 111111212, 111111213, 111111214, 111111215, 11111122, 11111123, 11111124, 11111125, 11111126, 11111127, 11111128, 11111129, 1111113, 11111131, 111111310, 111111311, 111111312, 111111313, 111111314, 111111315, 11111132, 11111133, 11111134, 11111135, 11111136, 11111137, 11111138, 11111139, 1111114, 1111115, 1111116, 1111117, 1111118, 1111119, 111112, 1111121, 11111210, 11111211, 11111212, 11111213, 11111214, 11111215, 1111122, 1111123, 1111124, 1111125, 1111126, 1111127, 1111128, 1111129, 111113, 11112, 111121, 111122, 111123, 11113, 111131, 111132, 111133, 11114, 111141, 111142, 111143, 11115, 111151, 111152, 111153, 11116, 11117, 1112, 11121, 11122, 11123, 11124, 11125, 11126, 11127, 1113, 11131, 11132, 11133, 11134, 11135, 11136, 11137, 1121, 1122, 1123, 1131, 1132, 1133: , ReST-Library:VIA-0.6mm
- removed ?: 1pin, ReST-Library:1pin
- removed G***: LOGO, ReST-Library:Logo_silk_OSHW_12x13mm
- removed G***: LOGO, ReST-Library:STM32-12mm
- removed P29, P31, P33: SCREW_01X03, 2:mpt_0,5%2f3-2,54
- removed REF** (x4): 1pin, Connect:1pin
- P23, P25, P27: value SCREW_01X03 -> CONN_01X06; footprint 2:mpt_0,5%2f3-2,54 -> 2:mpt_0,5%2f6-2,54
- U1: footprint ReST-Library:LQFP100-14x14 -> Housings_QFP:TQFP-100_14x14mm_Pitch0.5mm
- U3: footprint ReST-Library:SOT-404 -> TO_SOT_Packages_SMD:SOT-404
- moved P23 7.98 mm to (196.8, 114.0)
- moved P25 6.43 mm to (196.8, 130.2)
- moved P27 4.93 mm to (196.8, 146.2)
- turned U1 to 180 degrees
Routing:
- net (no net): track 0.00 -> 15.3 mm
- net GND: track 367.6 -> 352.7 mm
- net /ENDSTOP_VCC: track 92.3 -> 100.1 mm
- net /X-MIN: track 56.6 -> 58.4 mm
- net /X-MAX: track 48.2 -> 49.5 mm
- net /Y-MIN: track 55.7 -> 56.8 mm
- net /Y-MAX: track 57.7 -> 58.2 mm
