File: ReST Mainboard/ReST.sch (KiCad schematic (older format))
At the start: 79 parts, among them IC1 AT24C128, P1 CONN_01X03, P10 CONN_01X04, P11 CONN_01X04, P12 CONN_02X03, P14 CONN_02X03, P18 CONN_02X04, P19 CONN_01X04, P2 CONN_01X03, P21 CONN_02X04, P28 CONN_01X03, P3 CONN_01X03, P34 CONN_01X03, P35 SCREW_01X04, P36 SCREW_01X04, P37 SCREW_01X04, P38 SCREW_01X04, P39 CONN_02X04, P4 CONN_01X03, P40 CONN_01X04, P41 CONN_01X04, P42 CONN_01X04, P43 CONN_02X03, P44 CONN_02X03, P45 CONN_02X03, P46 CONN_02X03, P5 USB_OTG, P6 CONN_02X05, P7 CONN_02X05, P8 CONN_01X03, P9 CONN_01X02, SW1 SW-SPST-NO, U1 STM32F103VE, U2 USBLC6-2, U3 L7805ACD2T-TR, U4 LM3671MFX-3.3, U5 POLOLU_A4988, U6 POLOLU_A4988, U7 POLOLU_A4988, U8 POLOLU_A4988, X1 Crystal_Small

Commit message: Mainboard structure made and most modules finished
Parts:
- removed C10: 10uF, ReST-Library:CP-PANASONIC-SMT_C, symbol C_Small
- removed C11: 22uF, ReST-Library:CP-PANASONIC-SMT_D, symbol C_Small
- added C10: 10uF, ReST-Library:CP-PANASONIC-SMT_C, symbol CP1_Small
- added C11: 22uF, ReST-Library:CP-PANASONIC-SMT_D, symbol CP1_Small
- added D1: 1N400x, ReST-Library:DO-214AC.SMA, symbol D_Small
- added P13, P15: CONN_02X04, ReST-Library:REST_STEPPER, symbol CONN_02X04
- added P16: CONN_02X06, ReST-Library:REST_ADDITIONAL, symbol CONN_02X06
- added P17: CONN_02X03, ReST-Library:REST_HEATBED, symbol CONN_02X03
- added P23, P24: CONN_02X07, ReST-Library:REST_HEATER, symbol CONN_02X07
- added P27: CONN_02X06, Pin_Headers:Pin_Header_Straight_2x06, symbol CONN_02X06
- C7: footprint Capacitors_SMD:C_0805_HandSoldering -> Capacitors_SMD:C_0603_HandSoldering
- F1: footprint ReST-Library:JEF-703C -> ReST-Library:MINI-FUSE
- L2: footprint (none) -> ReST-Library:CD32
- P35, P36, P37, P38: footprint 2:mpt_0,5%2f4-2,54 -> ReST-Library:pt_1,5-4-3,5-h
- P43, P44, P45, P46: footprint Pin_Headers:Pin_Header_Straight_2x03 -> ReST-Library:bb02-hp06
- P8: footprint (none) -> Pin_Headers:Pin_Header_Straight_1x03
- P9: footprint 5mm-pitch-terminal:mkds_1,5-2 -> ReST-Library:screw-5-2P
- R2, R3: footprint Resistors_SMD:R_0805_HandSoldering -> Resistors_SMD:R_0603_HandSoldering
- U4: footprint SOT-23-5 -> TO_SOT_Packages_SMD:SOT-23-5
Connections:
- net +12V: now also C10.1, D1.1 (K), P13.7 (P7), P13.8 (P8), P15.7 (P7), P15.8 (P8), P16.10 (P10), P16.12 (P12), P16.6 (P6), P16.8 (P8), P23.5 (P5), P23.6 (P6), P23.7 (P7), P23.8 (P8), P23.9 (P9), P24.5 (P5), P24.6 (P6), P24.7 (P7), P24.8 (P8), P24.9 (P9)
- net +3V3: now also P13.5 (P5), P15.5 (P5), P17.2 (P2), P23.1 (P1), P24.1 (P1)
- net +5V: now also P17.1 (P1), P23.2 (P2), P24.2 (P2)
- net E1-DIR: now also P13.3 (P3)
- net E1-EN: now also P13.2 (P2)
- net E1-STEP: now also P13.1 (P1)
- net E2-DIR: now also P15.3 (P3)
- net E2-EN: now also P15.2 (P2)
- net E2-STEP: now also P15.1 (P1)
- net EXTRA0: now also P27.1 (P1)
- net EXTRA1: now also P27.2 (P2)
- net EXTRA10: now also P27.11 (P11)
- net EXTRA11: now also P27.12 (P12)
- net EXTRA2: now also P27.3 (P3)
- net EXTRA3: now also P27.4 (P4)
- net EXTRA4: now also P27.5 (P5)
- net EXTRA5: now also P27.6 (P6)
- net EXTRA6: now also P27.7 (P7)
- net EXTRA7: now also P27.8 (P8)
- net EXTRA8: now also P27.9 (P9)
- net EXTRA9: now also P27.10 (P10)
- net GND: now also C10.2, C11.2, D1.2 (A), P13.4 (P4), P13.6 (P6), P15.4 (P4), P15.6 (P6), P16.1 (P1), P16.2 (P2), P16.3 (P3), P16.4 (P4), P17.3 (P3), P17.5 (P5), P23.10 (P10), P23.11 (P11), P23.12 (P12), P23.13 (P13), P23.14 (P14), P24.10 (P10), P24.11 (P11), P24.12 (P12), P24.13 (P13), P24.14 (P14)
- net PWM-ADD0: now also P16.11 (P11)
- net PWM-ADD1: now also P16.9 (P9)
- net PWM-ADD2: now also P16.7 (P7)
- net PWM-ADD3: now also P16.5 (P5)
- net PWM-BED: now also P17.4 (P4)
- net PWM-HEAT0: now also P24.4 (P4)
- net PWM-HEAT1: now also P23.4 (P4)
- net T0: now also P17.6 (P6)
- net T1: now also P24.3 (P3)
- net T2: now also P23.3 (P3)
- net VEE: now also C11.1
- net at P40.4 (P4), U5.3 (IB): now also P36.1 (P1); no longer P36.4 (P4)
- net at P40.3 (P3), U5.4 (1A): now also P36.2 (P2); no longer P36.3 (P3)
- net at P40.2 (P2), U5.5 (2A): now also P36.3 (P3); no longer P36.2 (P2)
- net at P40.1 (P1), U5.6 (2B): now also P36.4 (P4); no longer P36.1 (P1)
- net at P41.4 (P4), U6.3 (IB): now also P37.1 (P1); no longer P37.4 (P4)
- net at P41.3 (P3), U6.4 (1A): now also P37.2 (P2); no longer P37.3 (P3)
- net at P41.2 (P2), U6.5 (2A): now also P37.3 (P3); no longer P37.2 (P2)
- net at P41.1 (P1), U6.6 (2B): now also P37.4 (P4); no longer P37.1 (P1)
- net at P39.1 (P1), P39.2 (P2), U7.3 (IB): now also P35.1 (P1); no longer P35.4 (P4)
- net at P39.3 (P3), P39.4 (P4), U7.4 (1A): now also P35.2 (P2); no longer P35.3 (P3)
- net at P39.5 (P5), P39.6 (P6), U7.5 (2A): now also P35.3 (P3); no longer P35.2 (P2)
- net at P39.7 (P7), P39.8 (P8), U7.6 (2B): now also P35.4 (P4); no longer P35.1 (P1)
- net at P42.4 (P4), U8.3 (IB): now also P38.1 (P1); no longer P38.4 (P4)
- net at P42.3 (P3), U8.4 (1A): now also P38.2 (P2); no longer P38.3 (P3)
- net at P42.2 (P2), U8.5 (2A): now also P38.3 (P3); no longer P38.2 (P2)
- net at P42.1 (P1), U8.6 (2B): now also P38.4 (P4); no longer P38.1 (P1)
Other:
- note added: "5V Rail\nUSB or EXT"
- note added: "Additional Output"
- note added: "Extra Pinout"
- note added: "Heatbed"
- note added: "Heater 1"
- note added: "Heater 2"
- note added: "Stepper 1"
- note added: "Stepper 2"
- note removed: "5V Rail\nUSB or REG"
- moved on the sheet: F1, IC1, P10, P11, P12, P14, P19, P9
