File: ReST Mainboard/ReST.sch (KiCad schematic (older format))
At the start: 87 parts, among them IC1 AT24C128, P1 CONN_01X03, P10 CONN_01X04, P11 CONN_01X04, P12 CONN_02X03, P13 CONN_02X04, P14 CONN_02X03, P15 CONN_02X04, P16 CONN_02X06, P17 CONN_02X03, P18 CONN_02X04, P19 CONN_01X04, P2 CONN_01X03, P21 CONN_02X04, P23 CONN_02X07, P24 CONN_02X07, P27 CONN_02X06, P28 CONN_01X03, P3 CONN_01X03, P34 CONN_01X03, P35 SCREW_01X04, P36 SCREW_01X04, P37 SCREW_01X04, P38 SCREW_01X04, P39 CONN_02X04, P4 CONN_01X03, P40 CONN_01X04, P41 CONN_01X04, P42 CONN_01X04, P43 CONN_02X03, P44 CONN_02X03, P45 CONN_02X03, P46 CONN_02X03, P5 USB_OTG, P6 CONN_02X05, P7 CONN_02X05, P8 CONN_01X03, P9 CONN_01X02, SW1 SW-SPST-NO, U1 STM32F103VE, U2 USBLC6-2, U3 L7805ACD2T-TR, U4 LM3671MFX-3.3, U5 POLOLU_A4988, U6 POLOLU_A4988, U7 POLOLU_A4988, U8 POLOLU_A4988, X1 Crystal_Small

Commit message: autosave
Connections:
- net E0-DIR: now also U1.78 (UART4_TX/SDIO_D2/PC10), U6.16 (DIR); no longer U1.87 (PD6/FSMC_NWAIT), U8.16 (DIR)
- net E0-EN: now also U1.80 (UART5_TX/SDIO_CK/PC12), U6.9 (EN); no longer U1.91 (I2C1_SMBA/SPI3_MOSI/I2S3_CD/PB5), U8.9 (EN)
- net E0-STEP: now also U1.79 (UART4_RX/SDIO_D3/PC11), U6.15 (STEP); no longer U1.88 (PD7/FSMC_NE1/FSMC_NCE2), U8.15 (STEP)
- net E1-DIR: now also U1.25 (USART2_TX/TIM5_CH3/ADC123_IN2/TIM2_CH3/PA2); no longer U1.18 (ADC123_IN13/PC3)
- net E1-EN: now also U1.29 (SPI1_NSS/USART2_CK/DAC_OUT1/ADC12_IN4/PA4); no longer U1.24 (USART2_RTS/ADC123_IN1/TIM5_CH2/TIM2_CH2/PA1)
- net E1-STEP: now also U1.26 (USART2_RX/TIM5_CH4/ADC123_IN3/TIM2_CH4/PA3); no longer U1.23 (WKUP/USART2_CTS/ADC123_IN0/TIM2_CH1_ETR/TIM5_CH1/TIM8_ETR/PA0)
- net E2-DIR: now also U1.18 (ADC123_IN13/PC3); no longer U1.25 (USART2_TX/TIM5_CH3/ADC123_IN2/TIM2_CH3/PA2)
- net E2-EN: now also U1.24 (USART2_RTS/ADC123_IN1/TIM5_CH2/TIM2_CH2/PA1); no longer U1.29 (SPI1_NSS/USART2_CK/DAC_OUT1/ADC12_IN4/PA4)
- net E2-STEP: now also U1.23 (WKUP/USART2_CTS/ADC123_IN0/TIM2_CH1_ETR/TIM5_CH1/TIM8_ETR/PA0); no longer U1.26 (USART2_RX/TIM5_CH4/ADC123_IN3/TIM2_CH4/PA3)
- net EXTRA10: now also U1.98 (PE1/FSMC_NBL1); no longer U1.82 (PD1/FSMC_D3)
- net EXTRA11: now also U1.1 (PE2/TRACECK/FSMC_A23); no longer U1.81 (PD0/FSMC_D2)
- net EXTRA4: now also U1.95 (TIM4_CH3/SDIO_D4/PB8); no longer U1.78 (UART4_TX/SDIO_D2/PC10)
- net EXTRA5: now also U1.96 (TIM4_CH4/SDIO_D5/PB9); no longer U1.79 (UART4_RX/SDIO_D3/PC11)
- net EXTRA8: now also U1.2 (PE3/TRACED0/FSMC_A19); no longer U1.80 (UART5_TX/SDIO_CK/PC12)
- net EXTRA9: now also U1.97 (PE0/TIM4_ETR/FSMC_NBL0); no longer U1.83 (PD2/TIM3_ETR/UART5_RX/SDIO_CMD)
- net I2C-SCL: now also R13.1; no longer R12.1
- net I2C-SDA: now also R12.1; no longer R13.1
- net X-DIR: now also U1.81 (PD0/FSMC_D2), U8.16 (DIR); no longer U1.98 (PE1/FSMC_NBL1), U5.16 (DIR)
- net X-EN: now also U1.83 (PD2/TIM3_ETR/UART5_RX/SDIO_CMD), U8.9 (EN); no longer U1.2 (PE3/TRACED0/FSMC_A19), U5.9 (EN)
- net X-STEP: now also U1.82 (PD1/FSMC_D3), U8.15 (STEP); no longer U1.1 (PE2/TRACECK/FSMC_A23), U5.15 (STEP)
- net Y-DIR: now also U1.84 (PD3/FSMC_CLK), U5.16 (DIR); no longer U1.95 (TIM4_CH3/SDIO_D4/PB8), U6.16 (DIR)
- net Y-EN: now also U1.86 (PD5/FSMC_NWE), U5.9 (EN); no longer U1.97 (PE0/TIM4_ETR/FSMC_NBL0), U6.9 (EN)
- net Y-STEP: now also U1.85 (PD4/FSMC_NOE), U5.15 (STEP); no longer U1.96 (TIM4_CH4/SDIO_D5/PB9), U6.15 (STEP)
- net Z-DIR: now also U1.91 (I2C1_SMBA/SPI3_MOSI/I2S3_CD/PB5); no longer U1.84 (PD3/FSMC_CLK)
- net Z-EN: now also U1.87 (PD6/FSMC_NWAIT); no longer U1.86 (PD5/FSMC_NWE)
- net Z-STEP: now also U1.88 (PD7/FSMC_NE1/FSMC_NCE2); no longer U1.85 (PD4/FSMC_NOE)
- net USB_D-: now reaches P5.2 (D-), U2.1 (I/O1)
- net USB_D+: now reaches P5.3 (D+), U2.3 (I/O2)
- net USBDM renamed USB-
- net USBDP renamed USB+
Other:
- moved on the sheet: R12, R13
Changed lines of the file:
@@
 	1    0    0    -1
 $EndComp
-Text Label 10600 2900 0    39   ~ 0
+Text Label 10650 6800 0    39   ~ 0
 X-DIR
-Text Label 10600 3000 0    39   ~ 0
+Text Label 10650 6900 0    39   ~ 0
 X-STEP
-Text Label 10600 3600 0    39   ~ 0
+Text Label 10650 7500 0    39   ~ 0
 X-EN
 $Comp
@@
 	-1   0    0    1
 $EndComp
-Text Label 10600 4900 0    39   ~ 0
+Text Label 10600 2900 0    39   ~ 0
 Y-DIR
-Text Label 10600 5000 0    39   ~ 0
+Text Label 10600 3000 0    39   ~ 0
 Y-STEP
-Text Label 10600 5600 0    39   ~ 0
+Text Label 10600 3600 0    39   ~ 0
 Y-EN
 $Comp
@@
 	-1   0    0    1
 $EndComp
-Text Label 10650 6800 0    39   ~ 0
+Text Label 10600 4900 0    39   ~ 0
 E0-DIR
-Text Label 10650 6900 0    39   ~ 0
+Text Label 10600 5000 0    39   ~ 0
 E0-STEP
-Text Label 10650 7500 0    39   ~ 0
+Text Label 10600 5600 0    39   ~ 0
 E0-EN
 $Comp
@@
 $EndComp
 Text Label 5000 5450 0    39   ~ 0
-USBDM
+USB-
 Text Label 5000 5550 0    39   ~ 0
-USBDP
+USB+
 Text Label 12350 1350 0    39   ~ 0
-USBDM
+USB-
 Text Label 12350 1250 0    39   ~ 0
-USBDP
+USB+
 $Comp
 L GND #PWR050
@@
 Text Label 2000 8650 2    39   ~ 0
 LCD-RD
-Text Label 5000 8950 0    39   ~ 0
+Text Label 2000 6350 2    39   ~ 0
 EXTRA8
-Text Label 2000 7950 2    39   ~ 0
+Text Label 2000 6050 2    39   ~ 0
 EXTRA9
 Text Label 5700 6650 0    39   ~ 0
@@
 Text Label 2000 6450 2    39   ~ 0
 Z-MAX
-Text Label 2000 6150 2    39   ~ 0
+Text Label 2000 7750 2    39   ~ 0
 X-DIR
-Text Label 2000 6250 2    39   ~ 0
+Text Label 2000 7850 2    39   ~ 0
 X-STEP
-Text Label 2000 6350 2    39   ~ 0
+Text Label 2000 7950 2    39   ~ 0
 X-EN
-Text Label 5000 6850 0    39   ~ 0
+Text Label 2000 8050 2    39   ~ 0
 Y-DIR
-Text Label 5000 6950 0    39   ~ 0
+Text Label 2000 8150 2    39   ~ 0
 Y-STEP
-Text Label 2000 6050 2    39   ~ 0
+Text Label 2000 8250 2    39   ~ 0
 Y-EN
-Text Label 2000 8050 2    39   ~ 0
+Text Label 5000 6550 0    39   ~ 0
 Z-DIR
-Text Label 2000 8150 2    39   ~ 0
+Text Label 2000 8450 2    39   ~ 0
 Z-STEP
-Text Label 2000 8250 2    39   ~ 0
-Z-EN
 Text Label 2000 8350 2    39   ~ 0
+Z-EN
+Text Label 5000 8750 0    39   ~ 0
 E0-DIR
-Text Label 2000 8450 2    39   ~ 0
+Text Label 5000 8850 0    39   ~ 0
 E0-STEP
-Text Label 5000 6550 0    39   ~ 0
+Text Label 5000 8950 0    39   ~ 0
 E0-EN
-Text Label 5000 8050 0    39   ~ 0
+Text Label 5000 4550 0    39   ~ 0
 E1-DIR
-Text Label 5000 4350 0    39   ~ 0
+Text Label 5000 4650 0    39   ~ 0
 E1-STEP
-Text Label 5000 4450 0    39   ~ 0
+Text Label 5000 4750 0    39   ~ 0
 E1-EN
-Text Label 5000 4550 0    39   ~ 0
+Text Label 5000 8050 0    39   ~ 0
 E2-DIR
-Text Label 5000 4650 0    39   ~ 0
+Text Label 5000 4350 0    39   ~ 0
 E2-STEP
-Text Label 5000 4750 0    39   ~ 0
+Text Label 5000 4450 0    39   ~ 0
 E2-EN
 Text Label 2000 9150 2    39   ~ 0
@@
 Text Label 5000 5150 0    39   ~ 0
 EXTRA3
-Text Label 5000 8750 0    39   ~ 0
+Text Label 5000 6850 0    39   ~ 0
 EXTRA4
-Text Label 5000 8850 0    39   ~ 0
+Text Label 5000 6950 0    39   ~ 0
 EXTRA5
 Text Label 2000 6750 2    39   ~ 0
@@
 L R_Small R12
 U 1 1 56D29E83
-P 5300 6550
-F 0 "R12" H 5330 6570 50  0000 L CNN
-F 1 "4K7" H 5330 6510 50  0000 L CNN
-F 2 "Resistors_SMD:R_0805_HandSoldering" H 5300 6550 50  0001 C CNN
-F 3 "" H 5300 6550 50  0000 C CNN
-	1    5300 6550
-	1    0    0    1
-$EndComp
-$Comp
-L R_Small R13
-U 1 1 56D2B222
 P 5500 6600
-F 0 "R13" H 5530 6620 50  0000 L CNN
+F 0 "R12" H 5530 6620 50  0000 L CNN
 F 1 "4K7" H 5530 6560 50  0000 L CNN
 F 2 "Resistors_SMD:R_0805_HandSoldering" H 5500 6600 50  0001 C CNN
@@
 $EndComp
 $Comp
+L R_Small R13
+U 1 1 56D2B222
+P 5300 6550
+F 0 "R13" H 5330 6570 50  0000 L CNN
+F 1 "4K7" H 5330 6510 50  0000 L CNN
+F 2 "Resistors_SMD:R_0805_HandSoldering" H 5300 6550 50  0001 C CNN
+F 3 "" H 5300 6550 50  0000 C CNN
+	1    5300 6550
+	1    0    0    1
+$EndComp
+$Comp
 L +3.3V #PWR077
 U 1 1 56D2CE65
@@
 	1    0    0    -1
 $EndComp
-Text Label 2000 7850 2    39   ~ 0
+Text Label 2000 6150 2    39   ~ 0
 EXTRA10
-Text Label 2000 7750 2    39   ~ 0
+Text Label 2000 6250 2    39   ~ 0
 EXTRA11
 $Comp
@@
 	13300 3550 13150 3550
 Connection ~ 13300 3450
+Text Label 10600 1250 0    39   ~ 0
+USB_D+
+Text Label 10550 1350 0    39   ~ 0
+USB_D-
 $EndSCHEMATC

Commit message: AUTOSAVE
Parts:
- P14: footprint Pin_Headers:Pin_Header_Straight_2x03 -> ReST-Library:bb02-hp06
- SW1: footprint Buttons_Switches_ThroughHole:SW_PUSH_SMALL -> ReST-Library:SMD-BUTTON-6MM
Connections:
- net +3V3: now also P10.2 (P2); no longer P11.2 (P2)
- net +5V: now also P11.1 (P1); no longer P10.1 (P1)
- net EXTRA2: no longer U1.66 (TIM8_CH4/SDIO_D1/PC9)
- net EXTRA3: no longer U1.67 (USART1_CK/TIM1_CH1/MCO/PA8)
- net GND: now also P10.1 (P1), P11.4 (P4); no longer P10.4 (P4), P11.1 (P1)
- net I2C-SCL: now also P10.4 (P4); no longer P11.3 (P3)
- net I2C-SDA: now also P10.3 (P3); no longer P11.4 (P4)
- net SWCLK: now also P19.3 (P3); no longer P10.3 (P3)
- net SWDIO: now also P19.2 (P2); no longer P10.2 (P2)
- net UART1-RX: now also P11.3 (P3); no longer P19.3 (P3)
- net UART1-TX: now also P11.2 (P2); no longer P19.2 (P2)
- no-connect marks 8 -> 10
Other:
- moved on the sheet: P10, P11, P19
Changed lines of the file:
@@
 Text Label 2000 9250 2    39   ~ 0
 EXTRA1
-Text Label 5000 8650 0    39   ~ 0
-EXTRA2
-Text Label 5000 5150 0    39   ~ 0
-EXTRA3
 Text Label 5000 6850 0    39   ~ 0
 EXTRA4
@@
 	1    0    0    -1
 $EndComp
+Text Label 14450 6550 2    39   ~ 0
+I2C-SCL
 Text Label 14450 6450 2    39   ~ 0
-I2C-SCL
-Text Label 14450 6550 2    39   ~ 0
 I2C-SDA
 Text Notes 14050 5850 0    39   ~ 0
@@
 L CONN_01X04 P10
 U 1 1 56CF969A
-P 15750 5100
-F 0 "P10" H 15750 5350 50  0000 C CNN
-F 1 "CONN_01X04" V 15850 5100 50  0000 C CNN
-F 2 "Pin_Headers:Pin_Header_Straight_1x04" H 15750 5100 50  0001 C CNN
-F 3 "" H 15750 5100 50  0000 C CNN
-	1    15750 5100
+P 14650 6400
+F 0 "P10" H 14650 6650 50  0000 C CNN
+F 1 "CONN_01X04" V 14750 6400 50  0000 C CNN
+F 2 "Pin_Headers:Pin_Header_Straight_1x04" H 14650 6400 50  0001 C CNN
+F 3 "" H 14650 6400 50  0000 C CNN
+	1    14650 6400
 	1    0    0    -1
 $EndComp
@@
 F 0 "SW1" H 1400 4350 60  0000 C CNN
 F 1 "SW-SPST-NO" H 1400 4150 60  0000 C CNN
-F 2 "Buttons_Switches_ThroughHole:SW_PUSH_SMALL" H 1400 4250 60  0001 C CNN
+F 2 "ReST-Library:SMD-BUTTON-6MM" H 1400 4250 60  0001 C CNN
 F 3 "" H 1400 4250 60  0000 C CNN
 	1    1400 4250
@@
 F 0 "P14" H 15450 6600 50  0000 C CNN
 F 1 "CONN_02X03" H 15450 6200 50  0000 C CNN
-F 2 "Pin_Headers:Pin_Header_Straight_2x03" H 15450 5200 50  0001 C CNN
+F 2 "ReST-Library:bb02-hp06" H 15450 5200 50  0001 C CNN
 F 3 "" H 15450 5200 50  0000 C CNN
 	1    15450 6400
@@
 L CONN_01X04 P11
 U 1 1 5735D1F0
-P 14650 6400
-F 0 "P11" H 14650 6650 50  0000 C CNN
-F 1 "CONN_01X04" V 14750 6400 50  0000 C CNN
-F 2 "Pin_Headers:Pin_Header_Straight_1x04" H 14650 6400 50  0001 C CNN
-F 3 "" H 14650 6400 50  0000 C CNN
-	1    14650 6400
+P 13150 8050
+F 0 "P11" H 13150 8300 50  0000 C CNN
+F 1 "CONN_01X04" V 13250 8050 50  0000 C CNN
+F 2 "Pin_Headers:Pin_Header_Straight_1x04" H 13150 8050 50  0001 C CNN
+F 3 "" H 13150 8050 50  0000 C CNN
+	1    13150 8050
 	1    0    0    -1
 $EndComp
@@
 L CONN_01X04 P19
 U 1 1 56CF54CA
-P 13150 8050
-F 0 "P19" H 13150 8300 50  0000 C CNN
-F 1 "CONN_01X04" V 13250 8050 50  0000 C CNN
-F 2 "Pin_Headers:Pin_Header_Straight_1x04" H 13150 8050 50  0001 C CNN
-F 3 "" H 13150 8050 50  0000 C CNN
-	1    13150 8050
+P 15750 5100
+F 0 "P19" H 15750 5350 50  0000 C CNN
+F 1 "CONN_01X04" V 15850 5100 50  0000 C CNN
+F 2 "Pin_Headers:Pin_Header_Straight_1x04" H 15750 5100 50  0001 C CNN
+F 3 "" H 15750 5100 50  0000 C CNN
+	1    15750 5100
 	1    0    0    -1
 $EndComp
@@
 Text Label 10550 1350 0    39   ~ 0
 USB_D-
+NoConn ~ 5000 8650
+NoConn ~ 5000 5150
 $EndSCHEMATC

Commit message: Rework. missing screws but everything else fits
Parts:
- removed P27: CONN_02X06, Pin_Headers:Pin_Header_Straight_2x06, symbol CONN_02X06
- removed SW1: SW-SPST-NO, ReST-Library:SMD-BUTTON-6MM, symbol SW-SPST-NO
- added P20, P22: CONN_02X04, ReST-Library:bb02-hp08, symbol CONN_02X04
- added S1: SW_DIP_x2, ReST-Library:SMD-BUTTON-6MM, symbol SW_DIP_x2
- C7: footprint Capacitors_SMD:C_0603_HandSoldering -> Capacitors_SMD:C_0805_HandSoldering
- P12: footprint Pin_Headers:Pin_Header_Straight_2x03 -> ReST-Library:bb02-hp06
- P6, P7: footprint Pin_Headers:Pin_Header_Straight_2x05 -> Connect:IDC_Header_Straight_10pins
- R2, R3: footprint Resistors_SMD:R_0603_HandSoldering -> Resistors_SMD:R_0805_HandSoldering
Connections:
- net +12V: now also P21.1 (P1), P21.3 (P3), P21.5 (P5), P21.7 (P7); no longer P18.1 (P1), P18.3 (P3), P18.5 (P5), P18.7 (P7)
- net +3V3: now also P10.4 (P4), P11.4 (P4), P18.2 (P2), P18.4 (P4), P18.6 (P6), P18.8 (P8), P19.4 (P4); no longer P10.2 (P2), P21.2 (P2), P21.4 (P4), P21.6 (P6), P21.8 (P8)
- net +5V: now also P18.1 (P1), P18.3 (P3), P18.5 (P5), P18.7 (P7); no longer P11.1 (P1), P19.1 (P1), P21.1 (P1), P21.3 (P3), P21.5 (P5), P21.7 (P7)
- net E0-DIR: now also U1.24 (USART2_RTS/ADC123_IN1/TIM5_CH2/TIM2_CH2/PA1), U5.16 (DIR); no longer U1.78 (UART4_TX/SDIO_D2/PC10), U6.16 (DIR)
- net E0-EN: now also U1.18 (ADC123_IN13/PC3), U5.9 (EN); no longer U1.80 (UART5_TX/SDIO_CK/PC12), U6.9 (EN)
- net E0-STEP: now also U1.23 (WKUP/USART2_CTS/ADC123_IN0/TIM2_CH1_ETR/TIM5_CH1/TIM8_ETR/PA0), U5.15 (STEP); no longer U1.79 (UART4_RX/SDIO_D3/PC11), U6.15 (STEP)
- net E1-DIR: now also U1.87 (PD6/FSMC_NWAIT); no longer U1.25 (USART2_TX/TIM5_CH3/ADC123_IN2/TIM2_CH3/PA2)
- net E1-EN: now also U1.91 (I2C1_SMBA/SPI3_MOSI/I2S3_CD/PB5); no longer U1.29 (SPI1_NSS/USART2_CK/DAC_OUT1/ADC12_IN4/PA4)
- net E1-STEP: now also U1.88 (PD7/FSMC_NE1/FSMC_NCE2); no longer U1.26 (USART2_RX/TIM5_CH4/ADC123_IN3/TIM2_CH4/PA3)
- net E2-DIR: now also U1.84 (PD3/FSMC_CLK); no longer U1.18 (ADC123_IN13/PC3)
- net E2-EN: now also U1.86 (PD5/FSMC_NWE); no longer U1.24 (USART2_RTS/ADC123_IN1/TIM5_CH2/TIM2_CH2/PA1)
- net E2-STEP: now also U1.85 (PD4/FSMC_NOE); no longer U1.23 (WKUP/USART2_CTS/ADC123_IN0/TIM2_CH1_ETR/TIM5_CH1/TIM8_ETR/PA0)
- net GND: now also P11.1 (P1), P19.1 (P1), P21.2 (P2), P21.4 (P4), P21.6 (P6), P21.8 (P8), P9.1 (P1), P20.7 (P7), P20.8 (P8), P22.7 (P7), P22.8 (P8), S1.3, S1.4; no longer P11.4 (P4), P18.2 (P2), P18.4 (P4), P18.6 (P6), P18.8 (P8), P19.4 (P4), P9.2 (P2)
- net I2C-SCL: now also P10.2 (P2); no longer P10.4 (P4)
- net LCD-CD: now also P7.9 (P9); no longer P7.1 (P1)
- net LCD-CS: now also P7.10 (P10); no longer P7.2 (P2)
- net LCD-D0: now also P7.2 (P2); no longer P7.10 (P10)
- net LCD-D1: now also P7.1 (P1); no longer P7.9 (P9)
- net LCD-D2: now also P7.4 (P4); no longer P7.8 (P8)
- net LCD-D3: now also P7.3 (P3); no longer P7.7 (P7)
- net LCD-D6: now also P7.8 (P8); no longer P7.4 (P4)
- net LCD-D7: now also P7.7 (P7); no longer P7.3 (P3)
- net PWM-ADD0: now also U1.36 (ADC12_IN9/TIM3_CH4/TIM8_CH3N/PB1); no longer U1.30 (SPI1_SCK/DAC_OUT2/ADC12_IN5/PA5)
- net PWM-ADD1: now also U1.63 (I2S2_MCK/TIM8_CH1/SDIO_D6/PC6); no longer U1.65 (TIM8_CH3/SDIO_D0/PC8)
- net PWM-ADD3: now also U1.65 (TIM8_CH3/SDIO_D0/PC8); no longer U1.63 (I2S2_MCK/TIM8_CH1/SDIO_D6/PC6)
- net PWM-BED: now also U1.31 (SPI1_MISO/TIM8_BKIN/ADC12_IN6/TIM3_CH1/PA6); no longer U1.36 (ADC12_IN9/TIM3_CH4/TIM8_CH3N/PB1)
- net PWM-HEAT1: now also U1.30 (SPI1_SCK/DAC_OUT2/ADC12_IN5/PA5); no longer U1.31 (SPI1_MISO/TIM8_BKIN/ADC12_IN6/TIM3_CH1/PA6)
- net RESET: now also S1.1, S1.2
- net T0: now also U1.33 (ADC12_IN14/PC4); no longer U1.35 (ADC12_IN8/TIM3_CH3/TIM8_CH2N/PB0)
- net T2: now also U1.35 (ADC12_IN8/TIM3_CH3/TIM8_CH2N/PB0); no longer U1.33 (ADC12_IN14/PC4)
- net UART1-RX: now also P11.2 (P2); no longer P11.3 (P3)
- net UART1-TX: now also P11.3 (P3); no longer P11.2 (P2)
- net VCC: now also P8.1 (P1); no longer P8.3 (P3)
- net VEE: now also P8.3 (P3); no longer P8.1 (P1)
- net X-DIR: now also U1.29 (SPI1_NSS/USART2_CK/DAC_OUT1/ADC12_IN4/PA4); no longer U1.81 (PD0/FSMC_D2)
- net X-EN: now also U1.25 (USART2_TX/TIM5_CH3/ADC123_IN2/TIM2_CH3/PA2); no longer U1.83 (PD2/TIM3_ETR/UART5_RX/SDIO_CMD)
- net X-MAX: now also U1.79 (UART4_RX/SDIO_D3/PC11); no longer U1.16 (ADC123_IN11/PC1)
- net X-MIN: now also U1.78 (UART4_TX/SDIO_D2/PC10); no longer U1.17 (ADC123_IN12/PC2)
- net X-STEP: now also U1.26 (USART2_RX/TIM5_CH4/ADC123_IN3/TIM2_CH4/PA3); no longer U1.82 (PD1/FSMC_D3)
- net Y-DIR: now also U1.15 (ADC123_IN10/PC0), U6.16 (DIR); no longer U1.84 (PD3/FSMC_CLK), U5.16 (DIR)
- net Y-EN: now also U1.17 (ADC123_IN12/PC2), U6.9 (EN); no longer U1.86 (PD5/FSMC_NWE), U5.9 (EN)
- net Y-MAX: now also U1.81 (PD0/FSMC_D2); no longer U1.5 (PE6/TRACED3/FSMC_A22)
- net Y-MIN: now also U1.80 (UART5_TX/SDIO_CK/PC12); no longer U1.15 (ADC123_IN10/PC0)
- net Y-STEP: now also U1.16 (ADC123_IN11/PC1), U6.15 (STEP); no longer U1.85 (PD4/FSMC_NOE), U5.15 (STEP)
- net Z-DIR: now also U1.3 (PE4/TRACED1/FSMC_A20); no longer U1.91 (I2C1_SMBA/SPI3_MOSI/I2S3_CD/PB5)
- net Z-EN: now also U1.5 (PE6/TRACED3/FSMC_A22); no longer U1.87 (PD6/FSMC_NWAIT)
- net Z-MAX: now also U1.83 (PD2/TIM3_ETR/UART5_RX/SDIO_CMD); no longer U1.3 (PE4/TRACED1/FSMC_A20)
- net Z-MIN: now also U1.82 (PD1/FSMC_D3); no longer U1.4 (PE5/TRACED2/FSMC_A21)
- net Z-STEP: now also U1.4 (PE5/TRACED2/FSMC_A21); no longer U1.88 (PD7/FSMC_NE1/FSMC_NCE2)
- net IO8: now reaches U1.66 (TIM8_CH4/SDIO_D1/PC9)
- net IO8: now also P22.2 (P2)
- net IO7: now reaches U1.67 (USART1_CK/TIM1_CH1/MCO/PA8)
- net IO7: now also P22.1 (P1)
- net USBR+: now reaches R2.1, U2.4 (I/O2)
- net USBR-: now reaches R3.2, U2.6 (I/O1)
- net 12V-RAW: now reaches F1.1
- net 12V-RAW: now also P9.2 (P2); no longer P9.1 (P1)
- net EXTRA0 renamed IO10
- net IO10: now also P22.4 (P4)
- net EXTRA1 renamed IO9
- net IO9: now also P22.3 (P3)
- net EXTRA10 renamed IO3
- net IO3: now also P20.3 (P3)
- net EXTRA11 renamed IO2
- net IO2: now also P20.2 (P2)
- net EXTRA4 renamed IO6
- net IO6: now also P20.6 (P6)
- net EXTRA5 renamed IO5
- net IO5: now also P20.5 (P5)
- net EXTRA6 renamed IO11
- net IO11: now also P22.5 (P5)
- net EXTRA7 renamed IO12
- net IO12: now also P22.6 (P6)
- net EXTRA8 renamed IO1
- net IO1: now also P20.1 (P1)
- net EXTRA9 renamed IO4
- net IO4: now also P20.4 (P4)
- no-connect marks 10 -> 8
Other:
- moved on the sheet: P18, P21

Commit message: Save of work
Parts:
- U3: footprint TO_SOT_Packages_SMD:SOT-404 -> ReST-Library:SOT-404
Changed lines of the file:
@@
 F 0 "U3" H 1250 1750 50  0000 C CNN
 F 1 "L7805ACD2T-TR" H 1450 1750 50  0000 L CNN
-F 2 "TO_SOT_Packages_SMD:SOT-404" H 1450 1650 50  0001 C CIN
+F 2 "ReST-Library:SOT-404" H 1450 1650 50  0001 C CIN
 F 3 "" H 1450 1550 50  0000 C CNN
 	1    1450 1550

Commit message: finishing touches on Heater and Stepper Modules
Parts:
- added P25: CONN_01X02, Pin_Headers:Pin_Header_Straight_1x02, symbol CONN_01X02
Connections:
- net GND: now also P25.2 (P2)
- net RESET: now also P25.1 (P1)
Other:
- note added: "Reset Pinout"
