File: ReST Mainboard/ReST.sch (KiCad schematic (older format))
At the start: 89 parts, among them IC1 AT24C128, P1 CONN_01X03, P10 CONN_01X04, P11 CONN_01X04, P12 CONN_02X03, P13 CONN_02X04, P14 CONN_02X03, P15 CONN_02X04, P16 CONN_02X06, P17 CONN_02X03, P18 CONN_02X04, P19 CONN_01X04, P2 CONN_01X03, P20 CONN_02X04, P21 CONN_02X04, P22 CONN_02X04, P23 CONN_02X07, P24 CONN_02X07, P25 CONN_01X02, P28 CONN_01X03, P3 CONN_01X03, P34 CONN_01X03, P35 SCREW_01X04, P36 SCREW_01X04, P37 SCREW_01X04, P38 SCREW_01X04, P39 CONN_02X04, P4 CONN_01X03, P40 CONN_01X04, P41 CONN_01X04, P42 CONN_01X04, P43 CONN_02X03, P44 CONN_02X03, P45 CONN_02X03, P46 CONN_02X03, P5 USB_OTG, P6 CONN_02X05, P7 CONN_02X05, P8 CONN_01X03, P9 CONN_01X02, U1 STM32F103VE, U2 USBLC6-2, U3 L7805ACD2T-TR, U4 LM3671MFX-3.3, U5 POLOLU_A4988, U6 POLOLU_A4988, U7 POLOLU_A4988, U8 POLOLU_A4988, X1 Crystal_Small

Commit message: Changes in Heatbed and Heater + F1 and F4 Pinout table with functions
Parts:
- removed P13, P15: CONN_02X04, ReST-Library:REST_STEPPER, symbol CONN_02X04
- removed U1: STM32F103VE, ReST-Library:LQFP100-14x14, symbol STM32F103VE
- added C? (x2): 100uF, ReST-Library:CP-PANASONIC-SMT_D8, symbol CP1_Small
- added C? (x2): 2.2uF, Capacitors_SMD:C_0805_HandSoldering, symbol C_Small
- added C?: 4.7uF, Capacitors_SMD:C_0805_HandSoldering, symbol C_Small
- added JP? (x2): JUMPER3, symbol JUMPER3
- added P? (x2): CONN_02X03, ReST-Library:bb02-hp06, symbol CONN_02X03
- added P? (x2): CONN_02X04, Pin_Headers:Pin_Header_Straight_2x04, symbol CONN_02X04
- added P? (x2): SCREW_01X04, ReST-Library:pt_1,5-4-3,5-h, symbol CONN_01X04
- added R? (x2): 100K, Resistors_SMD:R_0805_HandSoldering, symbol R_Small
- added U? (x2): POLOLU_A4988, ReST-Library:SWDIP8_.6W, symbol POLOLU_A4988
- added U?: STM32F10x/STM32F4x, ReST-Library:LQFP100-14x14, symbol STM32F10x/STM32F4x
Connections:
- net +12V: now also C?.1, C?.1, U?.8 (VMOT), U?.8 (VMOT)
- net +3V3: now also C?.1, JP?.1, P?.2 (P2), P?.2 (P2), P?.4 (P4), P?.4 (P4), P?.6 (P6), P?.6 (P6), U?.100 (VDD), U?.11 (VDD), U?.2 (VDD), U?.2 (VDD), U?.22 (VDDA), U?.28 (VDD), U?.50 (VDD), U?.75 (VDD)
- net BOOT0: now also U?.94 (BOOT0)
- net BOOT1: now also U?.37 (BOOT1/PB2)
- net E0-DIR: now also U?.24 (USART2_RTS/ADC123_IN1/TIM5_CH2/TIM2_CH2/PA1)
- net E0-EN: now also U?.18 (ADC123_IN13/PC3)
- net E0-STEP: now also U?.23 (WKUP/USART2_CTS/ADC123_IN0/TIM2_CH1_ETR/TIM5_CH1/TIM8_ETR/PA0)
- net E1-DIR: now also U?.87 (PD6/FSMC_NWAIT)
- net E1-EN: now also U?.91 (I2C1_SMBA/SPI3_MOSI/I2S3_CD/PB5)
- net E1-STEP: now also U?.88 (PD7/FSMC_NE1/FSMC_NCE2)
- net E2-DIR: now also U?.84 (PD3/FSMC_CLK)
- net E2-EN: now also U?.86 (PD5/FSMC_NWE)
- net E2-STEP: now also U?.85 (PD4/FSMC_NOE)
- net GND: now also C?.1, C?.2, C?.2, C?.2, C?.2, JP?.3, JP?.3, R?.2, R?.2, U?.1 (GND), U?.1 (GND), U?.10 (VSS), U?.20 (VREF-), U?.27 (VSS), U?.7 (GND), U?.7 (GND), U?.74 (VSS), U?.99 (VSS)
- net I2C-SCL: now also U?.92 (I2C1_SCL/TIM4_CH1/PB6)
- net I2C-SDA: now also U?.93 (I2C1_SDA/FSMC_NADV/TIM4_CH2/PB7)
- net IO1: now also U?.2 (PE3/TRACED0/FSMC_A19)
- net IO10: now also U?.61 (PD14/FSMC_D0)
- net IO11: now also U?.60 (PD13/FSMC_A18)
- net IO12: now also U?.59 (PD12/FSMC_A17)
- net IO2: now also U?.1 (PE2/TRACECK/FSMC_A23)
- net IO3: now also U?.98 (PE1/FSMC_NBL1)
- net IO4: now also U?.97 (PE0/TIM4_ETR/FSMC_NBL0)
- net IO5: now also U?.96 (TIM4_CH4/SDIO_D5/PB9)
- net IO6: now also U?.95 (TIM4_CH3/SDIO_D4/PB8)
- net IO7: now also U?.67 (USART1_CK/TIM1_CH1/MCO/PA8)
- net IO8: now also U?.66 (TIM8_CH4/SDIO_D1/PC9)
- net IO9: now also U?.62 (PD15/FSMC_D1)
- net LCD-CD: now also U?.47 (I2C2_SCL/USART3_TX/PB10)
- net LCD-CS: now also U?.46 (PE15/FSMC_D12)
- net LCD-D0: now also U?.38 (PE7/FSMC_D4)
- net LCD-D1: now also U?.39 (PE8/FSMC_D5)
- net LCD-D2: now also U?.40 (PE9/FSMC_D6)
- net LCD-D3: now also U?.41 (PE10/FSMC_D7)
- net LCD-D4: now also U?.42 (PE11/FSMC_D8)
- net LCD-D5: now also U?.43 (PE12/FSMC_D9)
- net LCD-D6: now also U?.44 (PE13/FSMC_D10)
- net LCD-D7: now also U?.45 (PE14/FSMC_D11)
- net LCD-RD: now also U?.56 (PD9/FSMC_D14)
- net LCD-WR: now also U?.48 (I2C2_SDA/USART3_RX/PB11)
- net PWM-ADD0: now also U?.36 (ADC12_IN9/TIM3_CH4/TIM8_CH3N/PB1)
- net PWM-ADD1: now also U?.63 (I2S2_MCK/TIM8_CH1/SDIO_D6/PC6)
- net PWM-ADD2: now also U?.64 (I2S3_MCK/TIM8_CH2/SDIO_D7/PC7)
- net PWM-ADD3: now also U?.65 (TIM8_CH3/SDIO_D0/PC8)
- net PWM-BED: now also U?.31 (SPI1_MISO/TIM8_BKIN/ADC12_IN6/TIM3_CH1/PA6)
- net PWM-HEAT0: now also U?.32 (SPI1_MOSI/TIM8_CH1N/ADC12_IN7/TIM3_CH2/PA7)
- net PWM-HEAT1: now also U?.30 (SPI1_SCK/DAC_OUT2/ADC12_IN5/PA5)
- net RESET: now also U?.14 (~NRST)
- net SERVO1: now also U?.57 (PD10/FSMC_D15)
- net SERVO2: now also U?.58 (PD11/FSMC_A16)
- net SPI-CS1: now also U?.51 (SPI2_NSS/I2S2_WS/I2C2_SMBA/USART3_CK/TIM1_BKIN/PB12)
- net SPI-CS2: now also U?.55 (PD8/FSMC_D13)
- net SPI-MISO: now also U?.53 (SPI2_MISO/TIM1_CH2N/USART3_RTS/PB14)
- net SPI-MOSI: now also U?.54 (SPI2_MOSI/I2S2_SD/TIM1_CH3N/PB15)
- net SPI-SCK: now also U?.52 (SPI2_SCK/I2S2_CK/USART3_CTS/TIM1_CH1N/PB13)
- net SWCLK: now also U?.76 (JTCK/SWCLK/PA14)
- net SWDIO: now also U?.72 (JTMS/SWDIO/PA13)
- net T0: now also U?.33 (ADC12_IN14/PC4)
- net T1: now also U?.34 (ADC12_IN15/PC5)
- net T2: now also U?.35 (ADC12_IN8/TIM3_CH3/TIM8_CH2N/PB0)
- net UART1-RX: now also U?.69 (USART1_RX/TIM1_CH3/PA10)
- net UART1-TX: now also U?.68 (USART1_TX/TIM1_CH2/PA9)
- net USB+: now also U?.71 (USART1_RTS/USBDP/CAN_TX/TIM1_ETR/PA11)
- net USB-: now also U?.70 (USART1_CTS/USBDM/CAN_RX/TIM1_CH4/PA11)
- net X-DIR: now also U?.29 (SPI1_NSS/USART2_CK/DAC_OUT1/ADC12_IN4/PA4)
- net X-EN: now also U?.25 (USART2_TX/TIM5_CH3/ADC123_IN2/TIM2_CH3/PA2)
- net X-MAX: now also U?.79 (UART4_RX/SDIO_D3/PC11)
- net X-MIN: now also U?.78 (UART4_TX/SDIO_D2/PC10)
- net X-STEP: now also U?.26 (USART2_RX/TIM5_CH4/ADC123_IN3/TIM2_CH4/PA3)
- net Y-DIR: now also U?.15 (ADC123_IN10/PC0)
- net Y-EN: now also U?.17 (ADC123_IN12/PC2)
- net Y-MAX: now also U?.81 (PD0/FSMC_D2)
- net Y-MIN: now also U?.80 (UART5_TX/SDIO_CK/PC12)
- net Y-STEP: now also U?.16 (ADC123_IN11/PC1)
- net Z-DIR: now also U?.16 (DIR), U?.16 (DIR), U?.3 (PE4/TRACED1/FSMC_A20)
- net Z-EN: now also U?.5 (PE6/TRACED3/FSMC_A22), U?.9 (EN), U?.9 (EN)
- net Z-MAX: now also U?.83 (PD2/TIM3_ETR/UART5_RX/SDIO_CMD)
- net Z-MIN: now also U?.82 (PD1/FSMC_D3)
- net Z-STEP: now also U?.15 (STEP), U?.15 (STEP), U?.4 (PE5/TRACED2/FSMC_A21)
- net at C24.2, X1.2: now also U?.12 (OSC_IN)
- net at C25.1, X1.1: now also U?.13 (OSC_OUT)
- net at C8.1, C9.1, L1.2: now also U?.21 (VREF+)
- new net: P?.1 (P1), R?.1, U?.10 (MS1) (x2)
- new net: P?.3 (P3), U?.11 (MS2) (x2)
- new net: P?.5 (P5), U?.12 (MS3) (x2)
- new net: U?.13 (RST), U?.14 (SLP) (x2)
- new net: P?.1 (P1), P?.1 (P1), P?.2 (P2), U?.3 (IB) (x2)
- new net: P?.2 (P2), P?.3 (P3), P?.4 (P4), U?.4 (1A) (x2)
- new net: P?.3 (P3), P?.5 (P5), P?.6 (P6), U?.5 (2A) (x2)
- new net: P?.4 (P4), P?.7 (P7), P?.8 (P8), U?.6 (2B) (x2)
- new net: JP?.2, U?.19 (VSSA)
- new net: C?.2, JP?.1
- new net: JP?.2, U?.49 (VSS)
- new net P73: C?.1, U?.73 (NC_/_VCAP_2)
Other:
- note added: "GND - F1\n3V3 - F4"
- note added: "GND - F1\nCAP - F4"
- note added: "Populate for F4"
- note added: "VDD3"
- note removed: "Stepper 1"
- note removed: "Stepper 2"
- moved on the sheet: C14, C15, C16, C17, C18, C19, C20, C21, C22, C23, C8, C9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

Commit message: temp push
Parts:
- removed C10: 10uF, ReST-Library:CP-PANASONIC-SMT_C, symbol CP1_Small
- removed C11: 22uF, ReST-Library:CP-PANASONIC-SMT_D, symbol CP1_Small
- removed C12, C13: 10uF, Capacitors_SMD:C_0805_HandSoldering, symbol C_Small
- removed C?: 100uF, ReST-Library:CP-PANASONIC-SMT_D8, symbol CP1_Small
- removed C? (x2): 2.2uF, Capacitors_SMD:C_0805_HandSoldering, symbol C_Small
- removed JP? (x2): JUMPER3, symbol JUMPER3
- removed P16: CONN_02X06, ReST-Library:REST_ADDITIONAL, symbol CONN_02X06
- removed P17: CONN_02X03, ReST-Library:REST_HEATBED, symbol CONN_02X03
- removed P18, P21, P? (x2): CONN_02X04, Pin_Headers:Pin_Header_Straight_2x04, symbol CONN_02X04
- removed P20, P22: CONN_02X04, ReST-Library:bb02-hp08, symbol CONN_02X04
- removed P23, P24: CONN_02X07, ReST-Library:REST_HEATER, symbol CONN_02X07
- removed P35, P36, P37, P38, P? (x2): SCREW_01X04, ReST-Library:pt_1,5-4-3,5-h, symbol CONN_01X04
- removed P43, P44, P45, P46, P? (x2): CONN_02X03, ReST-Library:bb02-hp06, symbol CONN_02X03
- removed R12, R13: 4K7, Resistors_SMD:R_0805_HandSoldering, symbol R_Small
- removed R?: 100K, Resistors_SMD:R_0805_HandSoldering, symbol R_Small
- removed U3: L7805ACD2T-TR, ReST-Library:SOT-404, symbol LM117H
- removed U4: LM3671MFX-3.3, TO_SOT_Packages_SMD:SOT-23-5, symbol LM3670MF
- removed U?: POLOLU_A4988, ReST-Library:SWDIP8_.6W, symbol POLOLU_A4988
- added C? (x4): 10uF, Capacitors_SMD:C_0805_HandSoldering, symbol C_Small
- added C? (x2): 2u2, Capacitors_SMD:C_0805_HandSoldering, symbol C_Small
- added C?: 22nF, Capacitors_SMD:C_0805_HandSoldering, symbol C_Small
- added C?: 4.7uF, Capacitors_SMD:C_0805_HandSoldering, symbol C_Small
- added D? (x4): 1N400x, ReST-Library:DO-214AC.SMA, symbol D_Small
- added D? (x3): Led_Small, symbol Led_Small
- added D?: B240A, symbol D_Schottky_Small
- added F?: F_Small, ReST-Library:MINI-FUSE, symbol F_Small
- added JP1: JUMPER3, ReST-Library:S_JUMPER_3, symbol JUMPER3
- added JP? (x2): JUMPER3, symbol JUMPER3
- added L?: 4.7uH, ReST-Library:CD32, symbol INDUCTOR_SMALL
- added P13, P18: CONN_02X03, Pin_Headers:Pin_Header_Straight_2x03, symbol CONN_02X03
- added P15: CONN_01X04, Pin_Headers:Pin_Header_Straight_1x04, symbol CONN_01X04
- added P? (x4): CONN_01X02, ReST-Library:screw-5-2P, symbol CONN_01X02
- added P? (x3): CONN_01X02, ReST-Library:bb02-hy02a, symbol CONN_01X02
- added P?: CONN_02X05, symbol CONN_02X05
- added Q? (x3): Q_BSH105/IRLML2502, ReST-Library:SOT-23, symbol Q_NMOS_GSD
- added Q? (x3): Q_AOT240L, ReST-Library:TO-220_Neutral123_Vertical_LargePads_Heatsink, symbol Q_NMOS_GSD
- added R? (x3): 4K7, Resistors_SMD:R_0603_HandSoldering, symbol R_Small
- added R? (x6): 100K, Resistors_SMD:R_0603_HandSoldering, symbol R_Small
- added R? (x3): 22R, Resistors_SMD:R_0603_HandSoldering, symbol R_Small
- added R? (x3): 150R, Resistors_SMD:R_0603_HandSoldering, symbol R_Small
- added R?: 28.7k, Resistors_SMD:R_0805_HandSoldering, symbol R_Small
- added R?: 150K, Resistors_SMD:R_0805_HandSoldering, symbol R_Small
- added R? (x2): 4K7, Resistors_SMD:R_0805_HandSoldering, symbol R_Small
- added U10: MCP23017, Housings_SSOP:SSOP-28_5.3x10.2mm_Pitch0.65mm, symbol MCP23017
- added U?: ACT4088, symbol ACT4088
- gave numbers to parts that had none: 5
Connections:
- net +12V: now also C?.1, D?.1 (K), D?.1 (K), P13.1 (P1), P13.3 (P3), P13.5 (P5), P?.2 (P2), P?.2 (P2), U?.2 (IN), U?.3 (EN)
- net +3V3: now also JP1.1, JP?.1, P18.2 (P2), P18.4 (P4), P18.6 (P6), R?.1, R?.1, R?.1, R?.2, R?.2, R?.2, R?.2, R?.2, U10.16 (A1), U10.17 (A2), U10.9 (VDD); no longer L2.2, P6.4 (P4)
- net +5V: now also P18.1 (P1), P18.3 (P3), P18.5 (P5), R?.1, R?.1, R?.1, R?.2, R?.2, R?.2
- net GND: now also C?.2, C?.2, C?.2, C?.2, C?.2, C?.2, C?.2, D?.2 (A), D?.2 (A), JP1.2, JP1.3, JP?.3, JP?.3, P13.2 (P2), P13.4 (P4), P13.6 (P6), P?.1 (P1), P?.1 (P1), P?.1 (P1), P?.1 (P1), Q?.2 (S), Q?.2 (S), Q?.2 (S), Q?.2 (S), Q?.2 (S), Q?.2 (S), R?.1, U10.10 (VSS), U10.15 (A0), U?.5 (GND)
- net I2C-SCL: now also U10.12 (SCL); no longer IC1.6 (SCL), P10.2 (P2), U1.92 (I2C1_SCL/TIM4_CH1/PB6)
- net I2C-SDA: now also U10.13 (SDA); no longer IC1.5 (SDA), P10.3 (P3), U1.93 (I2C1_SDA/FSMC_NADV/TIM4_CH2/PB7)
- net PWM-BED: now also Q?.1 (G), R?.1; no longer U1.31 (SPI1_MISO/TIM8_BKIN/ADC12_IN6/TIM3_CH1/PA6)
- net PWM-HEAT0: now also Q?.1 (G), R?.1; no longer U1.32 (SPI1_MOSI/TIM8_CH1N/ADC12_IN7/TIM3_CH2/PA7)
- net PWM-HEAT1: now also Q?.1 (G), R?.1; no longer U1.30 (SPI1_SCK/DAC_OUT2/ADC12_IN5/PA5)
- net T0: now also C?.1, P?.2 (P2), R?.2; no longer U1.33 (ADC12_IN14/PC4)
- net T1: now also C?.1, P?.2 (P2), R?.2; no longer U1.34 (ADC12_IN15/PC5)
- net T2: now also C?.1, P?.2 (P2), R?.2; no longer U1.35 (ADC12_IN8/TIM3_CH3/TIM8_CH2N/PB0)
- net VEE: now also C?.1, L?.2, R?.2
- net E0M1: now reaches R8.1, U5.10 (MS1)
- net E0M1: now also U10.24 (GPA3)
- net E0M2: now reaches U5.11 (MS2)
- net E0M2: now also U10.23 (GPA2)
- net E0M3: now reaches U5.12 (MS3)
- net E0M3: now also U10.22 (GPA1)
- net YM1: now reaches R9.1, U6.10 (MS1)
- net YM1: now also U10.6 (GPB5)
- net YM2: now reaches U6.11 (MS2)
- net YM2: now also U10.5 (GPB4)
- net YM3: now reaches U6.12 (MS3)
- net YM3: now also U10.4 (GPB3)
- net ZM1: now reaches R11.1, U7.10 (MS1)
- net ZM1: now also U10.21 (GPA0)
- net ZM2: now reaches U7.11 (MS2)
- net ZM2: now also U10.8 (GPB7)
- net ZM3: now reaches U7.12 (MS3)
- net ZM3: now also U10.7 (GPB6)
- net XM1: now reaches R10.1, U8.10 (MS1)
- net XM1: now also U10.3 (GPB2)
- net XM2: now reaches U8.11 (MS2)
- net XM2: now also U10.2 (GPB1)
- net XM3: now reaches U8.12 (MS3)
- net XM3: now also U10.1 (GPB0)
- net E1M1: now reaches R4.1, U9.10 (MS1)
- net E1M1: now also U10.27 (GPA6)
- net E1M2: now reaches U9.11 (MS2)
- net E1M2: now also U10.26 (GPA5)
- net E1M3: now reaches U9.12 (MS3)
- net E1M3: now also U10.25 (GPA4)
- net at U9.3 (IB): now also P15.4 (P4)
- net at U9.4 (1A): now also P15.3 (P3)
- net at U9.5 (2A): now also P15.2 (P2)
- net at U9.6 (2B): now also P15.1 (P1)
- net P_VSSA: now reaches U1.19 (VSSA)
- net P_VSSA: now also JP?.2
- net P_VCAP_1: now reaches U1.49 (VSS)
- net P_VCAP_1: now also JP?.2
- net DISPLAY_CD: now reaches U1.77 (JTDI/SPI3_NSS/I2S3_WS/PA15)
- net DISPLAY_CD: now also P7.9 (P9)
- net DISPLAY_WR: now reaches U1.89 (JTDO/SPI3_SCK/I2S3_CK/PB3)
- net DISPLAY_WR: now also P6.9 (P9)
- net BOOT0 renamed BOOT_0
- net BOOT1 renamed BOOT_1
- net E0-DIR renamed EXTRA_1
- net EXTRA_1: no longer U5.16 (DIR)
- net E0-EN renamed STEPPER_E_0_EN
- net STEPPER_E_0_EN: now also U1.57 (PD10/FSMC_D15); no longer U1.18 (ADC123_IN13/PC3)
- net E0-STEP renamed EXTRA_0
- net EXTRA_0: no longer U5.15 (STEP)
- net E1-DIR renamed DISPLAY_D6
- net DISPLAY_D6: now also P7.8 (P8)
- net E1-EN renamed DISPLAY_RD
- net DISPLAY_RD: now also P6.10 (P10)
- net E1-STEP renamed DISPLAY_D7
- net DISPLAY_D7: now also P7.7 (P7)
- net E2-DIR renamed DISPLAY_D3
- net DISPLAY_D3: now also P7.3 (P3)
- net E2-EN renamed DISPLAY_D5
- net DISPLAY_D5: now also P7.5 (P5)
- net E2-STEP renamed DISPLAY_D4
- net DISPLAY_D4: now also P7.6 (P6)
- net IO1 renamed ENDSTOP_Y_MIN
- net ENDSTOP_Y_MIN: now also C15.1, P2.3 (P3)
- net IO10 renamed STEPPER_E_1_STEP
- net STEPPER_E_1_STEP: now also U9.15 (STEP), U9.9 (EN)
- net IO11 renamed STEPPER_E_1_EN
- net IO12 renamed STEPPER_E_0_DIR
- net STEPPER_E_0_DIR: now also U5.16 (DIR)
- net IO2 renamed ENDSTOP_X_MAX
- net ENDSTOP_X_MAX: now also C17.1, P3.3 (P3)
- net IO3 renamed ENDSTOP_X_MIN
- net ENDSTOP_X_MIN: now also C14.1, P1.3 (P3)
- net IO4: no longer names the net of U1.97 (PE0/TIM4_ETR/FSMC_NBL0)
- net IO5 renamed DISPLAY_EXTRA_1
- net IO6 renamed DISPLAY_EXTRA_0
- net DISPLAY_EXTRA_0: now also P6.4 (P4)
- net IO7 renamed SERVO_1
- net SERVO_1: now also P12.2 (P2)
- net IO8 renamed SERVO_0
- net SERVO_0: now also P12.1 (P1)
- net IO9 renamed STEPPER_E_1_DIR
- net STEPPER_E_1_DIR: now also U9.16 (DIR)
- net LCD-CD renamed STEPPER_Z_STEP
- net STEPPER_Z_STEP: now also U7.15 (STEP); no longer P7.9 (P9)
- net LCD-CS renamed DISPLAY_CS
- net DISPLAY_CS: now also U1.80 (UART5_TX/SDIO_CK/PC12); no longer U1.46 (PE15/FSMC_D12)
- net LCD-D0 renamed DISPLAY_D0
- net DISPLAY_D0: now also U1.81 (PD0/FSMC_D2); no longer U1.38 (PE7/FSMC_D4)
- net LCD-D1 renamed DISPLAY_D1
- net DISPLAY_D1: now also U1.82 (PD1/FSMC_D3); no longer U1.39 (PE8/FSMC_D5)
- net LCD-D2 renamed DISPLAY_D2
- net DISPLAY_D2: now also U1.83 (PD2/TIM3_ETR/UART5_RX/SDIO_CMD); no longer U1.40 (PE9/FSMC_D6)
- net LCD-D3 renamed USER_3
- net USER_3: no longer P7.3 (P3)
- net LCD-D4 renamed USER_4
- net USER_4: no longer P7.6 (P6)
- net LCD-D5 renamed USER_5
- net USER_5: no longer P7.5 (P5)
- net LCD-D6 renamed USER_6
- net USER_6: no longer P7.8 (P8)
- net LCD-D7 renamed USER_7
- net USER_7: no longer P7.7 (P7)
- net LCD-RD renamed STEPPER_X_DIR
- net STEPPER_X_DIR: now also U8.16 (DIR); no longer P6.10 (P10)
- net LCD-WR renamed STEPPER_Z_DIR
- net STEPPER_Z_DIR: now also U7.16 (DIR); no longer P6.9 (P9)
- net P73 renamed P_VCAP_2
- net P_VCAP_2: now also C?.1
- net PWM-ADD0 renamed TEMP_5
- net PWM-ADD1 renamed HEATER_0
- net PWM-ADD2 renamed HEATER_1
- net PWM-ADD3 renamed HEATER_2
- removed net SERVO1: P12.1 (P1), U1.57 (PD10/FSMC_D15)
- net SERVO2 renamed STEPPER_E_0_STEP
- net STEPPER_E_0_STEP: now also U5.15 (STEP); no longer P12.2 (P2)
- net SPI-CS1 renamed SPI_CS1
- net SPI_CS1: now also U1.33 (ADC12_IN14/PC4); no longer U1.51 (SPI2_NSS/I2S2_WS/I2C2_SMBA/USART3_CK/TIM1_BKIN/PB12)
- net SPI-CS2 renamed SPI_CS2
- net SPI_CS2: now also U1.34 (ADC12_IN15/PC5); no longer U1.55 (PD8/FSMC_D13)
- net SPI-MISO renamed SPI_MISO
- net SPI_MISO: now also U1.31 (SPI1_MISO/TIM8_BKIN/ADC12_IN6/TIM3_CH1/PA6); no longer U1.53 (SPI2_MISO/TIM1_CH2N/USART3_RTS/PB14)
- net SPI-MOSI renamed SPI_MOSI
- net SPI_MOSI: now also U1.32 (SPI1_MOSI/TIM8_CH1N/ADC12_IN7/TIM3_CH2/PA7); no longer U1.54 (SPI2_MOSI/I2S2_SD/TIM1_CH3N/PB15)
- net SPI-SCK renamed SPI_SCK
- net SPI_SCK: now also U1.30 (SPI1_SCK/DAC_OUT2/ADC12_IN5/PA5); no longer U1.52 (SPI2_SCK/I2S2_CK/USART3_CTS/TIM1_CH1N/PB13)
- net SWCLK renamed SWD_CLK
- net SWDIO renamed SWD_IO
- net UART1-RX renamed UART_1_RX
- net UART1-TX renamed UART_1_TX
- net USB+ renamed USB_DP_+
- net USB- renamed USB_DM_-
- net X-DIR renamed SPI_CS0
- net SPI_CS0: no longer U8.16 (DIR)
- net X-EN renamed EXTRA_2
- net EXTRA_2: no longer U8.9 (EN)
- removed net X-MAX: C17.1, P3.3 (P3), U1.79 (UART4_RX/SDIO_D3/PC11)
- removed net X-MIN: C14.1, P1.3 (P3), U1.78 (UART4_TX/SDIO_D2/PC10)
- net X-STEP renamed EXTRA_3
- net EXTRA_3: no longer U8.15 (STEP)
- net Y-DIR renamed STEPPER_Y_DIR
- net STEPPER_Y_DIR: now also U1.53 (SPI2_MISO/TIM1_CH2N/USART3_RTS/PB14); no longer U1.15 (ADC123_IN10/PC0)
- net Y-EN renamed STEPPER_Y_EN
- net STEPPER_Y_EN: now also U1.51 (SPI2_NSS/I2S2_WS/I2C2_SMBA/USART3_CK/TIM1_BKIN/PB12); no longer U1.17 (ADC123_IN12/PC2)
- net Y-MAX renamed ENDSTOP_Y_MAX
- net ENDSTOP_Y_MAX: now also U1.3 (PE4/TRACED1/FSMC_A20); no longer U1.81 (PD0/FSMC_D2)
- removed net Y-MIN: C15.1, P2.3 (P3), U1.80 (UART5_TX/SDIO_CK/PC12)
- net Y-STEP renamed STEPPER_Y_STEP
- net STEPPER_Y_STEP: now also U1.52 (SPI2_SCK/I2S2_CK/USART3_CTS/TIM1_CH1N/PB13); no longer U1.16 (ADC123_IN11/PC1)
- removed net Z-DIR: U1.3 (PE4/TRACED1/FSMC_A20), U7.16 (DIR), U9.16 (DIR)
- removed net Z-EN: U1.5 (PE6/TRACED3/FSMC_A22), U7.9 (EN), U9.9 (EN)
- net Z-MAX renamed ENDSTOP_Z_MAX
- net ENDSTOP_Z_MAX: now also U1.5 (PE6/TRACED3/FSMC_A22); no longer U1.83 (PD2/TIM3_ETR/UART5_RX/SDIO_CMD)
- net Z-MIN renamed ENDSTOP_Z_MIN
- net ENDSTOP_Z_MIN: now also U1.4 (PE5/TRACED2/FSMC_A21); no longer U1.82 (PD1/FSMC_D3)
- removed net Z-STEP: U1.4 (PE5/TRACED2/FSMC_A21), U7.15 (STEP), U9.15 (STEP)
- new net: Q?.3 (D), R?.1, R?.1 (x3)
- new net: Q?.1 (G), R?.2 (x3)
- new net: D?.2 (A), R?.2 (x3)
- new net: C?.1, JP?.1
- new net: C?.1, D?.1 (K), L?.1, U?.1 (SW)
- new net: R?.1, R?.2, U?.4 (FB)
- new net: C?.2, U?.6 (BST)
- new net +12VA: D?.1 (K), D?.1 (K), F?.2, P?.2 (P2)
- new net H-12V-RAW: F?.1, P?.2 (P2)
- new net H1-MOS: D?.1 (K), D?.2 (A), P?.1 (P1), Q?.3 (D)
- new net H2-MOS: D?.1 (K), D?.2 (A), P?.1 (P1), Q?.3 (D)
- new net HB-MOS: D?.1 (K), D?.2 (A), P?.1 (P1), Q?.3 (D)
- new net I2C_SCL: IC1.6 (SCL), P10.2 (P2), R?.1, U1.92 (I2C1_SCL/TIM4_CH1/PB6)
- new net I2C_SDA: IC1.5 (SDA), P10.3 (P3), R?.1, U1.93 (I2C1_SDA/FSMC_NADV/TIM4_CH2/PB7)
- new net STEPPER_X_EN: U1.54 (SPI2_MOSI/I2S2_SD/TIM1_CH3N/PB15), U8.9 (EN)
- new net STEPPER_X_STEP: U1.55 (PD8/FSMC_D13), U8.15 (STEP)
- new net STEPPER_Z_EN: U1.46 (PE15/FSMC_D12), U7.9 (EN)
- new net TEMP_0: U1.15 (ADC123_IN10/PC0)
- new net TEMP_1: U1.16 (ADC123_IN11/PC1)
- new net TEMP_2: U1.17 (ADC123_IN12/PC2)
- new net TEMP_3: U1.18 (ADC123_IN13/PC3)
- new net TEMP_4: U1.35 (ADC12_IN8/TIM3_CH3/TIM8_CH2N/PB0)
- new net UART_4_RX: U1.79 (UART4_RX/SDIO_D3/PC11)
- new net UART_4_TX: U1.78 (UART4_TX/SDIO_D2/PC10)
- new net USER_0: U1.38 (PE7/FSMC_D4)
- new net USER_1: U1.39 (PE8/FSMC_D5)
- new net USER_2: U1.40 (PE9/FSMC_D6)
- no-connect marks 8 -> 11
Other:
- note added: "1-2 -> F4\n2-3 -> F1"
- note added: "2-1 and Cap -> F4\n2-3 and no Cap-> F1"
- note added: "Cap -> F4\nNo Cap -> F1"
- note added: "Heatbed PWR-IN"
- note added: "I2C Pullup"
- note added: "Power Supply Compability F1 and F4"
- note removed: "Additional Output"
- note removed: "GND - F1\n3V3 - F4"
- note removed: "GND - F1\nCAP - F4"
- note removed: "Heater 2"
- note removed: "Populate for F4"
- moved on the sheet: C14, C15, C16, C17, C18, C19, C20, C21, C22, C23, C27, C8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

Commit message: Hierarchical Schematic finished. Progress on PCB Layout
Parts:
- added C? (x2): 10uF, Capacitors_SMD:C_0805_HandSoldering, symbol C_Small
- added U?: SC4626, symbol SC4626
Connections:
- wire segments 455 -> 466
Other:
- moved on the sheet: L2
Changed lines of the file:
@@
 Text Notes 14350 4600 0    39   ~ 0
 EEPROM
-Text Notes 2700 950  0    39   ~ 0
+Text Notes 2300 -750 0    39   ~ 0
 VIN -> 3.3V BUCK CONVERTER
 NoConn ~ 10450 1450
@@
 L +3.3V #PWR074
 U 1 1 57355CED
-P 4400 1350
-F 0 "#PWR074" H 4400 1200 50  0001 C CNN
-F 1 "+3.3V" H 4400 1490 50  0000 C CNN
-F 2 "" H 4400 1350 50  0000 C CNN
-F 3 "" H 4400 1350 50  0000 C CNN
-	1    4400 1350
+P 4400 -500
+F 0 "#PWR074" H 4400 -650 50  0001 C CNN
+F 1 "+3.3V" H 4400 -360 50  0000 C CNN
+F 2 "" H 4400 -500 50  0000 C CNN
+F 3 "" H 4400 -500 50  0000 C CNN
+	1    4400 -500
 	1    0    0    -1
 $EndComp
@@
 L INDUCTOR_SMALL L2
 U 1 1 57355F82
-P 4000 1450
-F 0 "L2" H 4000 1550 50  0000 C CNN
-F 1 "2.2uH" H 4000 1400 50  0000 C CNN
-F 2 "ReST-Library:CD32" H 4000 1450 50  0001 C CNN
-F 3 "" H 4000 1450 50  0000 C CNN
-	1    4000 1450
+P 3950 -400
+F 0 "L2" H 3950 -300 50  0000 C CNN
+F 1 "2.2uH" H 3950 -450 50  0000 C CNN
+F 2 "ReST-Library:CD32" H 3950 -400 50  0001 C CNN
+F 3 "" H 3950 -400 50  0000 C CNN
+	1    3950 -400
 	1    0    0    -1
 $EndComp
@@
 L GND #PWR075
 U 1 1 5735961A
-P 3400 1900
-F 0 "#PWR075" H 3400 1650 50  0001 C CNN
-F 1 "GND" H 3400 1750 50  0000 C CNN
-F 2 "" H 3400 1900 50  0000 C CNN
-F 3 "" H 3400 1900 50  0000 C CNN
-	1    3400 1900
+P 4400 0
+F 0 "#PWR075" H 4400 -250 50  0001 C CNN
+F 1 "GND" H 4400 -150 50  0000 C CNN
+F 2 "" H 4400 0   50  0000 C CNN
+F 3 "" H 4400 0   50  0000 C CNN
+	1    4400 0
 	1    0    0    -1
 $EndComp
@@
 L GND #PWR076
 U 1 1 57359FA3
-P 2900 1900
-F 0 "#PWR076" H 2900 1650 50  0001 C CNN
-F 1 "GND" H 2900 1750 50  0000 C CNN
-F 2 "" H 2900 1900 50  0000 C CNN
-F 3 "" H 2900 1900 50  0000 C CNN
-	1    2900 1900
-	1    0    0    -1
-$EndComp
-$Comp
-L GND #PWR077
-U 1 1 5735A0AA
-P 4400 1900
-F 0 "#PWR077" H 4400 1650 50  0001 C CNN
-F 1 "GND" H 4400 1750 50  0000 C CNN
-F 2 "" H 4400 1900 50  0000 C CNN
-F 3 "" H 4400 1900 50  0000 C CNN
-	1    4400 1900
+P 2550 -100
+F 0 "#PWR076" H 2550 -350 50  0001 C CNN
+F 1 "GND" H 2550 -250 50  0000 C CNN
+F 2 "" H 2550 -100 50  0000 C CNN
+F 3 "" H 2550 -100 50  0000 C CNN
+	1    2550 -100
 	1    0    0    -1
 $EndComp
@@
 L +5V #PWR091
 U 1 1 57369D13
-P 2900 1350
-F 0 "#PWR091" H 2900 1200 50  0001 C CNN
-F 1 "+5V" H 2900 1490 50  0000 C CNN
-F 2 "" H 2900 1350 50  0000 C CNN
-F 3 "" H 2900 1350 50  0000 C CNN
-	1    2900 1350
+P 2550 -500
+F 0 "#PWR091" H 2550 -650 50  0001 C CNN
+F 1 "+5V" H 2550 -360 50  0000 C CNN
+F 2 "" H 2550 -500 50  0000 C CNN
+F 3 "" H 2550 -500 50  0000 C CNN
+	1    2550 -500
 	1    0    0    -1
 $EndComp
@@
 	10650 1450 10550 1450
 Wire Notes Line
-	5000 2350 5000 800
-Wire Notes Line
-	2350 2350 5000 2350
-Wire Notes Line
-	2350 800  2350 2350
-Wire Notes Line
-	5000 800  2350 800
-Wire Notes Line
 	13950 5650 13950 4500
 Wire Notes Line
@@
 Wire Notes Line
 	-3300 450  -3300 -1050
+$Comp
+L SC4626 U?
+U 1 1 576E98F0
+P 3250 -300
+F 0 "U?" H 3450 -100 39  0000 C CNN
+F 1 "SC4626" H 3100 -100 39  0000 C CNN
+F 2 "" H 3250 -300 39  0000 C CNN
+F 3 "" H 3250 -300 39  0000 C CNN
+	1    3250 -300
+	1    0    0    -1
+$EndComp
+$Comp
+L C_Small C?
+U 1 1 576EE934
+P 4400 -200
+F 0 "C?" H 4410 -130 50  0000 L CNN
+F 1 "10uF" H 4410 -280 50  0000 L CNN
+F 2 "Capacitors_SMD:C_0805_HandSoldering" H 4400 -200 50  0001 C CNN
+F 3 "" H 4400 -200 50  0000 C CNN
+	1    4400 -200
+	1    0    0    -1
+$EndComp
+Wire Wire Line
+	4200 -400 4400 -400
+Wire Wire Line
+	3700 -200 4250 -200
+Wire Wire Line
+	4250 -200 4250 -400
+Connection ~ 4250 -400
+Wire Wire Line
+	4400 -500 4400 -300
+Connection ~ 4400 -400
+Wire Wire Line
+	4400 0    4400 -100
+$Comp
+L C_Small C?
+U 1 1 576F49DB
+P 2550 -300
+F 0 "C?" H 2560 -230 50  0000 L CNN
+F 1 "10uF" H 2560 -380 50  0000 L CNN
+F 2 "Capacitors_SMD:C_0805_HandSoldering" H 2550 -300 50  0001 C CNN
+F 3 "" H 2550 -300 50  0000 C CNN
+	1    2550 -300
+	-1   0    0    1
+$EndComp
+Wire Wire Line
+	2800 -400 2550 -400
+Wire Wire Line
+	2550 -400 2550 -500
+Wire Wire Line
+	2800 -200 2550 -200
+Wire Wire Line
+	2800 -300 2700 -300
+Wire Wire Line
+	2700 -300 2700 -400
+Connection ~ 2700 -400
+Wire Wire Line
+	2550 -200 2550 -100
+Wire Notes Line
+	2300 -700 4650 -700
+Wire Notes Line
+	4650 -700 4650 200
+Wire Notes Line
+	4650 200  2300 200
+Wire Notes Line
+	2300 200  2300 -700
 $EndSCHEMATC
