File: ReST Mainboard/ReST.kicad_pcb (KiCad board)
At the start: 2 copper layers, 100 x 100 mm, 201 parts, among them U1 STM32F103VE

Commit message: finishing touches on Heater and Stepper Modules
Parts:
- added ?: , ReST-Library:1pin, F.Cu at (147.8, 111.0)
- added ?: , ReST-Library:1pin, F.Cu at (147.6, 114.4)
- added ?: , ReST-Library:1pin, F.Cu at (159.9, 127.7)
- added ?: , ReST-Library:1pin, F.Cu at (154.0, 127.8)
- added ?: , ReST-Library:1pin, F.Cu at (138.1, 116.3)
- added ?: , ReST-Library:1pin, F.Cu at (188.1, 121.3)
- added ?: , ReST-Library:1pin, F.Cu at (192.2, 120.3)
- added P25: , Pin_Headers:Pin_Header_Straight_1x02, F.Cu at (140.6, 126.7)
- C1, C2, C3, C4, C5, C6, C7, C9: value (none) -> 100nF
- C12, C13, C8: value (none) -> 10uF
- C14, C15, C16, C17, C18, C19: value (none) -> 10nF
- C24, C25: value (none) -> 30pF
- D1: value (none) -> 1N400x
- F1: renamed from Mini Fuse; value (none) -> F_Small
- IC1: value (none) -> AT24C128
- L1: value (none) -> BEAD
- L2: value (none) -> 2.2uH
- P1, P2, P28, P3, P34, P4, P8: renamed from ?; value (none) -> CONN_01X03
- P10, P11, P19, P40, P41, P42: renamed from ?; value (none) -> CONN_01X04
- P12, P14, P17, P43, P44, P45, P46: renamed from ?; value (none) -> CONN_02X03
- P13, P15, P18, P20, P21, P39: renamed from ?; value (none) -> CONN_02X04
- P16: renamed from ?; value (none) -> CONN_02X06
- P22: value (none) -> CONN_02X04
- P23, P24: renamed from ?; value (none) -> CONN_02X07
- P35, P36, P37, P38: renamed from ?; value (none) -> SCREW_01X04
- P5: renamed from ?; value (none) -> USB_OTG
- P6, P7: value (none) -> CONN_02X05
- P9: renamed from ?; value (none) -> CONN_01X02
- R1: value (none) -> 1M
- R10, R11, R8, R9: value (none) -> 100K
- R12, R13: value (none) -> 4K7
- R2, R3: value (none) -> 22R
- R5: value (none) -> 10K
- S1: value (none) -> SW_DIP_x2
- U2: value (none) -> USBLC6-2
- U3: value (none) -> L7805ACD2T-TR
- U4: value (none) -> LM3671MFX-3.3
- U5, U6, U7, U8: renamed from ?; value (none) -> POLOLU_A4988
- X1: value (none) -> Crystal_Small
- moved R8 2.47 mm to (172.2, 139.9)
- moved C20 2.39 mm to (172.2, 145.0)
- moved U5 2.17 mm to (172.9, 138.8)
- moved P36 2.17 mm to (172.9, 156.2)
- moved P40 2.15 mm to (169.1, 150.6)
- moved P43 2.14 mm to (172.6, 134.5)
- moved R10 1.55 mm to (156.8, 139.9)
- moved C23 1.43 mm to (156.8, 145.0)
- moved P46 1.30 mm to (157.2, 134.5)
- moved U8 1.19 mm to (157.5, 138.8)
- moved P38 1.19 mm to (157.5, 156.2)
- moved P42 1.18 mm to (153.7, 150.6)
- moved R9 1.00 mm to (141.1, 139.9)
- moved P45 0.98 mm to (125.8, 131.9)
- moved P44 0.90 mm to (141.5, 134.5)
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Routing:
- net +12V: track 243.0 -> 159.4 mm
- net +3V3: track 498.1 -> 414.5 mm
- net Net-(P35-Pad1): track 29.4 -> 0.00 mm
- net Net-(P37-Pad1): track 27.1 -> 0.00 mm
- net Net-(P38-Pad1): track 27.0 -> 0.00 mm
- net Net-(P36-Pad1): track 26.9 -> 0.00 mm
- net Net-(P35-Pad2): track 25.1 -> 0.00 mm
- net Net-(P37-Pad2): track 22.8 -> 0.00 mm
- net Net-(P38-Pad2): track 22.7 -> 0.00 mm
- net Net-(P36-Pad2): track 22.6 -> 0.00 mm
- net Net-(P35-Pad3): track 21.2 -> 0.00 mm
- net /Z-EN: track 56.0 -> 35.2 mm
- net /X-EN: track 40.7 -> 20.6 mm
- net /Y-EN: track 53.2 -> 33.8 mm
- net Net-(P37-Pad3): track 18.8 -> 0.00 mm
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Other:
- rule pad_to_mask_clearance: 0.2 -> 0

Commit message: minor changes
Parts:
- removed the ? at (133.7, 122.2)
- removed the ? at (191.8, 151.4)
- removed the ? at (188.1, 121.3)
- removed the ? at (192.2, 120.3)
- added 111: , ReST-Library:1pin, F.Cu at (114.0, 80.0)
- added 1111: , ReST-Library:1pin, F.Cu at (106.0, 80.0)
- added 1112: , ReST-Library:1pin, F.Cu at (106.0, 81.5)
- added 1113: , ReST-Library:1pin, F.Cu at (106.0, 83.0)
- added 1114: , ReST-Library:1pin, F.Cu at (106.0, 84.5)
- added 1115: , ReST-Library:1pin, F.Cu at (106.0, 86.0)
- added 1116: , ReST-Library:1pin, F.Cu at (106.0, 87.5)
- added 1117: , ReST-Library:1pin, F.Cu at (106.0, 89.0)
- added 1118: , ReST-Library:1pin, F.Cu at (106.0, 90.5)
- added 1119: , ReST-Library:1pin, F.Cu at (106.0, 92.0)
- added 112: , ReST-Library:1pin, F.Cu at (114.0, 81.5)
- added 1121: , ReST-Library:1pin, F.Cu at (107.5, 80.0)
- added 1122: , ReST-Library:1pin, F.Cu at (107.5, 81.5)
- added 1123: , ReST-Library:1pin, F.Cu at (107.5, 83.0)
- added 1124: , ReST-Library:1pin, F.Cu at (107.5, 84.5)
- added 1125: , ReST-Library:1pin, F.Cu at (107.5, 86.0)
- added 1126: , ReST-Library:1pin, F.Cu at (107.5, 87.5)
- added 1127: , ReST-Library:1pin, F.Cu at (107.5, 89.0)
- added 1128: , ReST-Library:1pin, F.Cu at (107.5, 90.5)
- added 1129: , ReST-Library:1pin, F.Cu at (107.5, 92.0)
- added 113: , ReST-Library:1pin, F.Cu at (114.0, 83.0)
- added 1131: , ReST-Library:1pin, F.Cu at (109.0, 80.0)
- added 1132: , ReST-Library:1pin, F.Cu at (109.0, 81.5)
- added 1133: , ReST-Library:1pin, F.Cu at (109.0, 83.0)
- added 1134: , ReST-Library:1pin, F.Cu at (109.0, 84.5)
- added 1135: , ReST-Library:1pin, F.Cu at (109.0, 86.0)
- added 1136: , ReST-Library:1pin, F.Cu at (109.0, 87.5)
- added 1137: , ReST-Library:1pin, F.Cu at (109.0, 89.0)
- added 1138: , ReST-Library:1pin, F.Cu at (109.0, 90.5)
- added 1139: , ReST-Library:1pin, F.Cu at (109.0, 92.0)
- added 114: , ReST-Library:1pin, F.Cu at (114.0, 84.5)
- added 1141: , ReST-Library:1pin, F.Cu at (110.5, 80.0)
- added 1142: , ReST-Library:1pin, F.Cu at (110.5, 81.5)
- added 1143: , ReST-Library:1pin, F.Cu at (110.5, 83.0)
- added 1144: , ReST-Library:1pin, F.Cu at (110.5, 84.5)
- added 1145: , ReST-Library:1pin, F.Cu at (110.5, 86.0)
- added 1146: , ReST-Library:1pin, F.Cu at (110.5, 87.5)
- added 1147: , ReST-Library:1pin, F.Cu at (110.5, 89.0)
- added 1148: , ReST-Library:1pin, F.Cu at (110.5, 90.5)
- added 1149: , ReST-Library:1pin, F.Cu at (110.5, 92.0)
- added 115: , ReST-Library:1pin, F.Cu at (114.0, 86.0)
- added 1151: , ReST-Library:1pin, F.Cu at (112.0, 80.0)
- added 1152: , ReST-Library:1pin, F.Cu at (112.0, 81.5)
- added 1153: , ReST-Library:1pin, F.Cu at (112.0, 83.0)
- added 1154: , ReST-Library:1pin, F.Cu at (112.0, 84.5)
- added 1155: , ReST-Library:1pin, F.Cu at (112.0, 86.0)
- added 1156: , ReST-Library:1pin, F.Cu at (112.0, 87.5)
- added 1157: , ReST-Library:1pin, F.Cu at (112.0, 89.0)
- added 1158: , ReST-Library:1pin, F.Cu at (112.0, 90.5)
- added 1159: , ReST-Library:1pin, F.Cu at (112.0, 92.0)
- added 116: , ReST-Library:1pin, F.Cu at (114.0, 87.5)
- added 117: , ReST-Library:1pin, F.Cu at (114.0, 89.0)
- added 118: , ReST-Library:1pin, F.Cu at (114.0, 90.5)
- added 119: , ReST-Library:1pin, F.Cu at (114.0, 92.0)
- added 121: , ReST-Library:1pin, F.Cu at (115.5, 80.0)
- added 122: , ReST-Library:1pin, F.Cu at (115.5, 81.5)
- added 123: , ReST-Library:1pin, F.Cu at (115.5, 83.0)
- added 124: , ReST-Library:1pin, F.Cu at (115.5, 84.5)
- added 125: , ReST-Library:1pin, F.Cu at (115.5, 86.0)
- added 126: , ReST-Library:1pin, F.Cu at (115.5, 87.5)
- added 127: , ReST-Library:1pin, F.Cu at (115.5, 89.0)
- added 128: , ReST-Library:1pin, F.Cu at (115.5, 90.5)
- added 129: , ReST-Library:1pin, F.Cu at (115.5, 92.0)
- added 131: , ReST-Library:1pin, F.Cu at (117.0, 80.0)
- added 132: , ReST-Library:1pin, F.Cu at (117.0, 81.5)
- added 133: , ReST-Library:1pin, F.Cu at (117.0, 83.0)
- added 134: , ReST-Library:1pin, F.Cu at (117.0, 84.5)
- added 135: , ReST-Library:1pin, F.Cu at (117.0, 86.0)
- added 136: , ReST-Library:1pin, F.Cu at (117.0, 87.5)
- added 137: , ReST-Library:1pin, F.Cu at (117.0, 89.0)
- added 138: , ReST-Library:1pin, F.Cu at (117.0, 90.5)
- added 139: , ReST-Library:1pin, F.Cu at (117.0, 92.0)
- added 141: , ReST-Library:1pin, F.Cu at (118.5, 80.0)
- added 142: , ReST-Library:1pin, F.Cu at (118.5, 81.5)
- added 143: , ReST-Library:1pin, F.Cu at (118.5, 83.0)
- added 144: , ReST-Library:1pin, F.Cu at (118.5, 84.5)
- added 145: , ReST-Library:1pin, F.Cu at (118.5, 86.0)
- added 146: , ReST-Library:1pin, F.Cu at (118.5, 87.5)
- added 147: , ReST-Library:1pin, F.Cu at (118.5, 89.0)
- added 148: , ReST-Library:1pin, F.Cu at (118.5, 90.5)
- added 149: , ReST-Library:1pin, F.Cu at (118.5, 92.0)
- added 151: , ReST-Library:1pin, F.Cu at (120.0, 80.0)
- added 152: , ReST-Library:1pin, F.Cu at (120.0, 81.5)
- added 153: , ReST-Library:1pin, F.Cu at (120.0, 83.0)
- added 154: , ReST-Library:1pin, F.Cu at (120.0, 84.5)
- added 155: , ReST-Library:1pin, F.Cu at (120.0, 86.0)
- added 156: , ReST-Library:1pin, F.Cu at (120.0, 87.5)
- added 157: , ReST-Library:1pin, F.Cu at (120.0, 89.0)
- added 158: , ReST-Library:1pin, F.Cu at (120.0, 90.5)
- added 159: , ReST-Library:1pin, F.Cu at (120.0, 92.0)
- added 161: , ReST-Library:1pin, F.Cu at (121.5, 80.0)
- added 162: , ReST-Library:1pin, F.Cu at (121.5, 81.5)
- added 163: , ReST-Library:1pin, F.Cu at (121.5, 83.0)
- added 164: , ReST-Library:1pin, F.Cu at (121.5, 84.5)
- added 165: , ReST-Library:1pin, F.Cu at (121.5, 86.0)
- added 166: , ReST-Library:1pin, F.Cu at (121.5, 87.5)
- added 167: , ReST-Library:1pin, F.Cu at (121.5, 89.0)
- added 168: , ReST-Library:1pin, F.Cu at (121.5, 90.5)
- added 169: , ReST-Library:1pin, F.Cu at (121.5, 92.0)
- added ?: , ReST-Library:1pin, F.Cu at (154.7, 120.1)
- added ?: , ReST-Library:1pin, F.Cu at (199.9, 94.2)
- added ?: , ReST-Library:1pin, F.Cu at (199.9, 92.7)
- added ?: , ReST-Library:1pin, F.Cu at (198.4, 92.7)
- added ?: , ReST-Library:1pin, F.Cu at (196.9, 92.7)
- added ?: , ReST-Library:1pin, F.Cu at (196.9, 91.2)
- added ?: , ReST-Library:1pin, F.Cu at (199.9, 91.2)
- added ?: , ReST-Library:1pin, F.Cu at (198.4, 91.2)
- added ?: , ReST-Library:1pin, F.Cu at (198.4, 89.7)
- added ?: , ReST-Library:1pin, F.Cu at (188.5, 108.7)
- added ?: , ReST-Library:1pin, F.Cu at (199.8, 112.0)
- added ?: , ReST-Library:1pin, F.Cu at (183.1, 151.2)
- added ?: , ReST-Library:1pin, F.Cu at (181.2, 151.8)
- added ?: , ReST-Library:1pin, F.Cu at (188.2, 152.1)
- added ?: , ReST-Library:1pin, F.Cu at (190.3, 152.1)
- added ?: , ReST-Library:1pin, F.Cu at (192.1, 151.2)
- added ?: , ReST-Library:1pin, F.Cu at (157.7, 117.3)
- added ?: , ReST-Library:1pin, F.Cu at (198.4, 94.2)
- ?: renamed from P1; value CONN_01X03 -> (none)
- ?: renamed from P3; value CONN_01X03 -> (none)
- ?: renamed from P4; value CONN_01X03 -> (none)
- ?: renamed from P28; value CONN_01X03 -> (none)
- ?: renamed from P34; value CONN_01X03 -> (none)
- ?: renamed from P2; value CONN_01X03 -> (none)
- P7: value CONN_02X05 -> (none)
- moved ? 7.92 mm to (119.5, 74.0)
- moved ? 2.30 mm to (199.9, 89.7)
- moved ? 2.30 mm to (194.7, 158.4)
- moved ? 2.30 mm to (192.1, 158.4)
- moved ? 2.30 mm to (184.5, 158.4)
- moved ? 2.30 mm to (182.0, 158.4)
- moved ? 2.30 mm to (187.0, 158.4)
- moved ? 2.30 mm to (189.6, 158.4)
- moved ? 1.50 mm to (200.4, 155.4)
- moved ? 1.34 mm to (196.1, 133.1)
- moved ? 1.26 mm to (196.4, 150.4)
- moved P39 1.14 mm to (128.8, 148.4)
- moved C20 1.09 mm to (173.2, 145.1)
- moved C21 0.99 mm to (142.1, 145.1)
- moved C23 0.89 mm to (157.7, 145.1)
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Routing:
- net +3V3: track 414.5 -> 512.5 mm, vias 8 -> 10
- net +12V: track 159.4 -> 227.6 mm
- net Net-(P35-Pad1): track 0.00 -> 29.8 mm
- net Net-(P37-Pad1): track 0.00 -> 28.0 mm
- net Net-(P38-Pad1): track 0.00 -> 27.6 mm
- net Net-(P36-Pad1): track 0.00 -> 27.6 mm
- net Net-(P35-Pad2): track 0.00 -> 25.5 mm
- net Net-(P38-Pad2): track 0.00 -> 23.5 mm
- net Net-(P37-Pad2): track 0.00 -> 23.0 mm
- net Net-(P36-Pad2): track 0.00 -> 22.7 mm
- net Net-(P35-Pad3): track 0.00 -> 21.5 mm
- net /Z-EN: track 35.2 -> 56.1 mm, vias 1 -> 3
- net /LCD-RD: track 33.6 -> 54.4 mm
- net Net-(P38-Pad3): track 0.00 -> 19.8 mm
- net Net-(P36-Pad3): track 0.00 -> 19.3 mm
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Other:
- board text removed: "X+"
- board text removed: "Y+"
- board text removed: "Y-"
- board text removed: "Z+"
- board text removed: "Z-"

Commit message: temp push
Parts:
- removed 111, 1111, 1112, 1113, 1114, 1115, 1116, 1117, 1118, 1119, 112, 1121, 1122, 1123, 1124, 1125, 1126, 1127, 1128, 1129, 113, 1131, 1132, 1133, 1134, 1135, 1136, 1137, 1138, 1139, 114, 1141, 1142, 1143, 1144, 1145, 1146, 1147, 1148, 1149, 115, 1151, 1152, 1153, 1154, 1155, 1156, 1157, 1158, 1159, 116, 117, 118, 119, 121, 122, 123, 124, 125, 126, 127, 128, 129, 131, 132, 133, 134, 135, 136, 137, 138, 139, 141, 142, 143, 144, 145, 146, 147, 148, 149, 151, 152, 153, 154, 155, 156, 157, 158, 159, 161, 162, 163, 164, 165, 166, 167, 168, 169, ? (x133): , ReST-Library:1pin
- removed ? (x6): , Pin_Headers:Pin_Header_Straight_1x03
- removed G***: LOGO, ReST-Library:NG3DC
- removed P21: CONN_02X04, Pin_Headers:Pin_Header_Straight_2x04
- removed P35, P36, P37, P38: SCREW_01X04, ReST-Library:pt_1,5-4-3,5-h
- removed P43, P44, P45, P46: CONN_02X03, ReST-Library:bb02-hp06
- added C26: 4.7uF, Capacitors_SMD:C_0805_HandSoldering, F.Cu at (96.0, 78.8)
- added C27: 100uF, ReST-Library:CP-PANASONIC-SMT_D8, F.Cu at (144.8, 123.3)
- added JP1: JUMPER3, ReST-Library:S_JUMPER_3, F.Cu at (163.8, 96.2)
- added P1: CONN_01X03, Pin_Headers:Pin_Header_Straight_1x03, F.Cu at (156.8, 70.2)
- added P2: CONN_01X03, Pin_Headers:Pin_Header_Straight_1x03, F.Cu at (168.4, 70.0)
- added P28: CONN_01X03, Pin_Headers:Pin_Header_Straight_1x03, F.Cu at (170.9, 89.5)
- added P3: CONN_01X03, Pin_Headers:Pin_Header_Straight_1x03, F.Cu at (178.3, 79.2)
- added P34: CONN_01X03, Pin_Headers:Pin_Header_Straight_1x03, F.Cu at (139.8, 109.2)
- added P4: CONN_01X03, Pin_Headers:Pin_Header_Straight_1x03, F.Cu at (171.8, 103.2)
- added R4: 100K, Resistors_SMD:R_0805_HandSoldering, F.Cu at (177.8, 73.7)
- added U10: MCP23017, Housings_SSOP:SSOP-28_5.3x10.2mm_Pitch0.65mm, F.Cu at (125.3, 115.3)
- added U9: POLOLU_A4988, ReST-Library:SWDIP8_.6W, F.Cu at (64.2, 152.2)
- P13: value CONN_02X04 -> CONN_02X03; footprint ReST-Library:REST_STEPPER -> Pin_Headers:Pin_Header_Straight_2x03
- P15: value CONN_02X04 -> CONN_01X04; footprint ReST-Library:REST_STEPPER -> Pin_Headers:Pin_Header_Straight_1x04
- P18: value CONN_02X04 -> CONN_02X03; footprint Pin_Headers:Pin_Header_Straight_2x04 -> Pin_Headers:Pin_Header_Straight_2x03
- P25: value (none) -> CONN_01X02
- P7: value (none) -> CONN_02X05
- U1: value STM32F103VE -> STM32F10x/STM32F4x
- moved P16 136.0 mm to (60.5, 78.0), turned to 0 degrees
- moved U6 106.5 mm to (35.9, 127.8), turned to 0 degrees
- moved C17 104.4 mm to (116.8, 66.5), turned to 0 degrees
- moved P17 103.4 mm to (222.8, 76.7)
- moved C12 102.1 mm to (195.2, 83.0), turned to 0 degrees
- moved U5 101.9 mm to (72.0, 124.5), turned to 0 degrees
- moved P23 93.9 mm to (251.3, 104.7)
- moved P40 92.2 mm to (100.0, 89.5), turned to 0 degrees
- moved C13 90.9 mm to (177.3, 70.8), turned to 0 degrees
- moved C18 90.9 mm to (123.8, 87.3), turned to 0 degrees
- moved P18 90.0 mm to (144.6, 71.5), turned to 0 degrees
- moved P24 86.1 mm to (216.9, 122.2)
- moved P7 85.8 mm to (189.8, 61.4), turned to 0 degrees
- moved P5 84.7 mm to (189.7, 95.3)
- moved C19 83.3 mm to (109.5, 113.8), turned to 0 degrees
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Connections:
- net Net-(P43-Pad1) renamed /E0M1
- net Net-(P44-Pad1) renamed /YM1
- net Net-(P45-Pad1) renamed /ZM1
- net Net-(P46-Pad1) renamed /XM1
- P13 pad 1: /E1-STEP -> +12V
- P13 pad 2: /E1-EN -> GND
- P13 pad 3: /E1-DIR -> +12V
- P13 pad 5: +3V3 -> +12V
- P15 pad 1: /E2-STEP -> Net-(P15-Pad1)
- P15 pad 2: /E2-EN -> Net-(P15-Pad2)
- P15 pad 3: /E2-DIR -> Net-(P15-Pad3)
- P15 pad 4: GND -> Net-(P15-Pad4)
- P20 pad 3: /IO3 -> (no net)
- P20 pad 4: /IO4 -> (no net)
- P20 pad 6: /IO6 -> (no net)
- P6 pad 4: +3V3 -> /LCD_PWM
- U1 pad 84: /E2-DIR -> /XRST
- U1 pad 85: /E2-STEP -> /YRST
- U1 pad 86: /E2-EN -> /ZRST
- U1 pad 95: /IO6 -> /LCD_PWM
- U1 pad 97: /IO4 -> /E0RST
- U1 pad 98: /IO3 -> /E1RST
- U5 pad 11: Net-(P43-Pad3) -> /E0M2
- U5 pad 12: Net-(P43-Pad5) -> /E0M3
- U5 pad 13: Net-(U5-Pad13) -> /E0RST
- U5 pad 14: Net-(U5-Pad13) -> /E0RST
- U6 pad 11: Net-(P44-Pad3) -> /YM2
- U6 pad 12: Net-(P44-Pad5) -> /YM3
- U6 pad 13: Net-(U6-Pad13) -> /YRST
- U6 pad 14: Net-(U6-Pad13) -> /YRST
- U7 pad 11: Net-(P45-Pad3) -> /ZM2
- U7 pad 12: Net-(P45-Pad5) -> /ZM3
- U7 pad 13: Net-(U7-Pad13) -> /ZRST
- U7 pad 14: Net-(U7-Pad13) -> /ZRST
- U8 pad 11: Net-(P46-Pad3) -> /XM2
- U8 pad 12: Net-(P46-Pad5) -> /XM3
- U8 pad 13: Net-(U8-Pad13) -> /XRST
- U8 pad 14: Net-(U8-Pad13) -> /XRST
Routing:
- net +3V3: track 512.5 -> 0.00 mm, vias 10 -> 0
- net +5V: track 232.7 -> 0.00 mm, vias 8 -> 0
- net +12V: track 227.6 -> 0.00 mm, vias 2 -> 0
- net GND: track 139.3 -> 0.00 mm, vias 5 -> 0
- net /PWM-HEAT1: track 88.1 -> 0.00 mm, vias 3 -> 0
- net /X-MIN: track 78.7 -> 0.00 mm, vias 2 -> 0
- net /T2: track 77.7 -> 0.00 mm, vias 3 -> 0
- net /X-MAX: track 77.4 -> 0.00 mm, vias 2 -> 0
- net /USB-: track 76.2 -> 0.00 mm, vias 2 -> 0
- net /Y-MIN: track 74.3 -> 0.00 mm, vias 2 -> 0
- net /USB+: track 74.3 -> 0.00 mm, vias 2 -> 0
- net /Y-MAX: track 72.8 -> 0.00 mm, vias 1 -> 0
- net /Z-MIN: track 72.0 -> 0.00 mm, vias 1 -> 0
- net /Z-MAX: track 71.3 -> 0.00 mm, vias 1 -> 0
- net /PWM-BED: track 70.5 -> 0.00 mm, vias 3 -> 0
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- removed copper zone on B.Cu, net +12V
- removed copper zone on F.Cu, net +12V
- removed copper zone on B.Cu, net /12V-RAW
- removed copper zone on F.Cu, net /12V-RAW
- removed copper zone on B.Cu, net GND
- removed copper zone on F.Cu, net GND
Other:
- board outline removed
- board text removed: "12V"
- board text removed: "2 ounce board!"
- board text removed: "3.3V"
- board text removed: "5V"
- board text removed: "5V Selector USB - REG"
- board text removed: "Additional High Power Module"
- board text removed: "COLORED Pinheaders! BLUE BLACK RED"
- board text removed: "E0 Stepper"
- board text removed: "E1 Stepper Module"
- board text removed: "E2 Stepper Module"
- board text removed: "GND"
- board text removed: "Heatbed Module"
- board text removed: "Heater 1 Module"
- board text removed: "Heater 2 Module"
- board text removed: "Next Gen 3D Printer Controller"
- board text removed: "X Stepper"
- board text removed: "X-"
- board text removed: "Y Stepper"
- board text removed: "Z Stepper"
