File: ReST-SD-Module/ReST SD-Module.sch (KiCad schematic (older format))
At the start: 7 parts, among them CON1 uSD_Card, CON2 uSD_Card, P1 CONN_02X05, U1 MIC5205

Commit message: minor changes to values of components and footprints. added two leds for both 12V Rails.
Parts:
- D1: footprint LEDs:LED_1206 -> LEDs:LED_0805
Changed lines of the file:
@@
 F 0 "D1" H 3750 3925 50  0000 L CNN
 F 1 "Led_Small" H 3625 3700 50  0000 L CNN
-F 2 "LEDs:LED_1206" V 3800 3800 50  0001 C CNN
+F 2 "LEDs:LED_0805" V 3800 3800 50  0001 C CNN
 F 3 "" V 3800 3800 50  0000 C CNN
 	1    3800 3800
